Commit message: add stl and velodyne urdf

File: src/rove_description/urdf/lidar.urdf.xacro (robot description, xacro)
@@ -2,56 +2,7 @@
 <robot xmlns:xacro="http://www.ros.org/wiki/xacro">
     <xacro:property name="M_PI" value="3.1415926535897931" />
-    <joint name="laser_joint" type="fixed">
-        <parent link="base_link"/>
-        <child link="base_scan"/>
-      <origin xyz="0.0 0 0.4" rpy="0 0 0"/>
-    </joint>
-    <link name="base_scan">
-        <visual>
-            <geometry>
-                <cylinder radius="0.05" length="0.04"/>
-            </geometry>
-        </visual>
-        <collision>
-            <geometry>
-                <cylinder radius="0.05" length="0.04"/>
-            </geometry>
-        </collision>
-        <inertial>
-            <origin xyz="0 0 0" rpy="0 0 0"/>
-            <mass value="0.1" />
-            <inertia ixx="${(1/12) * 0.1 * (3*0.05*0.05 + 0.04*0.04)}" ixy="0.0" ixz="0.0"
-                     iyy="${(1/12) * 0.1 * (3*0.05*0.05 + 0.04*0.04)}" iyz="0.0"
-                     izz="${(1/2) * 0.1 * (0.05*0.05)}" />
-        </inertial>
-    </link>
-    <gazebo reference="base_scan">
-        <material>Gazebo/Black</material>
-        <sensor name='laser_sensor_frame' type='gpu_lidar'>
-            <pose> 0 0 0 0 0 0 </pose>
-            <visualize>true</visualize>
-            <always_on>true</always_on>
-            <update_rate>5</update_rate>
-            <topic>scan</topic>
-            <gz_frame_id>base_scan</gz_frame_id>
-            <ray>
-                <scan>
-                    <horizontal>
-                        <samples>360</samples>
-                        <min_angle>-3.14</min_angle>
-                        <max_angle>3.14</max_angle>
-                    </horizontal>
-                </scan>
-                <range>
-                    <min>1</min>
-                    <max>50</max>
-                </range>
-                <noise>
-                    <type>gaussian</type>
-                    <mean>0.0</mean>
-                    <stddev>0.007</stddev>
-                </noise>
-            </ray>
-        </sensor>
-    </gazebo>
+    <xacro:include filename="$(find rove_description)/urdf/velodyne.urdf.xacro" />
+    <xacro:velodyne_lidar name="velodyne" parent_link="base_link">
+        <origin xyz="0.0 0.0 0.4" rpy="0 0 0" />
+    </xacro:velodyne_lidar>
 </robot>

File: src/rove_description/urdf/velodyne.urdf.xacro (robot description, xacro)
@@ -1,5 +1,4 @@
 <?xml version="1.0"?>
 <robot xmlns:xacro="http://www.ros.org/wiki/xacro">
-  <xacro:include filename="$(find velodyne_description)/urdf/VLP-16.urdf.xacro" />
   <xacro:macro name="velodyne_lidar" params="name parent_link *origin
                                              ang_res_h:=0.4 min_ang_h:=-3.141592 max_ang_h:=3.141592
@@ -19,10 +18,10 @@
       <visual>
         <geometry>
-          <mesh filename="package://velodyne_description/meshes/VLP16_base_1.dae"/>
+          <mesh filename="file://$(find rove_description)/meshes/vlp16/VLP16_base_1.dae"/>
         </geometry>
       </visual>
       <visual>
         <geometry>
-          <mesh filename="package://velodyne_description/meshes/VLP16_base_2.dae"/>
+          <mesh filename="file://$(find rove_description)/meshes/vlp16/VLP16_base_2.dae"/>
         </geometry>
       </visual>
@@ -48,5 +47,5 @@
         <origin xyz="0 0 -0.0377"/>
         <geometry>
-          <mesh filename="package://velodyne_description/meshes/VLP16_scan.dae"/>
+          <mesh filename="file://$(find rove_description)/meshes/vlp16/VLP16_scan.dae"/>
         </geometry>
       </visual>
@@ -64,5 +63,7 @@
         <visualize>true</visualize>
         <always_on>true</always_on>
-        <ignition_frame_id>${name}_laser</ignition_frame_id>
+        <update_rate>5</update_rate>
+        <topic>scan</topic>
+        <gz_frame_id>${name}_laser</gz_frame_id>
         <lidar>
           <scan>
