Commit message: remove track mass

File: src/rove_description/urdf/track.urdf.xacro (robot description, xacro)
@@ -21,7 +21,4 @@
             <parent link="track_${suffix}"/>
             <child link="track_f${suffix}"/>
-            <!-- <axis xyz="0 1 0"/>
-            <dynamics damping="0.2"/>
-            <limit effort="100" velocity="1.0"/> -->
         </joint>
         <joint name="track_r${suffix}_j" type="fixed">
@@ -29,7 +26,4 @@
             <parent link="track_${suffix}"/>
             <child link="track_r${suffix}"/>
-            <!-- <axis xyz="0 -1 0"/>
-            <dynamics damping="0.2"/>
-            <limit effort="100" velocity="1.0"/> -->
         </joint>
         <link name="track_${suffix}">
@@ -69,6 +63,4 @@
             <inertial>
                 <origin xyz="0 0 0" rpy="0 0 0"/>
-                <mass value="1"/>
-                <inertia ixx="100"  ixy="0"  ixz="0" iyy="100" iyz="0" izz="100" />
             </inertial>
         </link>
@@ -76,6 +68,4 @@
             <inertial>
                 <origin xyz="0 0 0" rpy="0 0 0"/>
-                <mass value="1"/>
-                <inertia ixx="100"  ixy="0"  ixz="0" iyy="100" iyz="0" izz="100" />
             </inertial>
         </link>
