Commit message: Not quite stable

File: src/rove_description/urdf/rove.ros2_control.urdf.xacro (robot description, xacro)
@@ -19,5 +19,5 @@
             </hardware>
             <joint name="track_fr_j">
-                <param name="node_id">23</param>
+                <param name="node_id">19</param>
                 <command_interface name="velocity"/>
                 <state_interface name="position"/>
@@ -54,10 +54,10 @@
             <xacro:rove_odrive_motor position="r" suffix="r" id="${rr_id}"/> -->
         </ros2_control>
-        <ros2_control name="fake_odrive_control" type="system">
+        <!-- <ros2_control name="fake_odrive_control" type="system">
             <hardware>
                 <plugin>mock_components/GenericSystem</plugin>
                 <param name="calculate_dynamics">true</param>
             </hardware>
-            <!-- <joint name="track_fl_j">
+            <<joint name="track_fl_j">
                 <param name="node_id">1</param>
                 <command_interface name="velocity"/>
@@ -72,6 +72,6 @@
                 <state_interface name="velocity"/>
                 <state_interface name="effort"/>
-            </joint> -->
-            <!-- <joint name="track_fr_j">
+            </joint>
+            <joint name="track_fr_j">
                 <param name="node_id">3</param>
                 <command_interface name="velocity"/>
@@ -86,6 +86,6 @@
                 <state_interface name="velocity"/>
                 <state_interface name="effort"/>
-            </joint> -->
-        </ros2_control>
+            </joint>
+        </ros2_control> -->
         <!-- <ros2_control name="fake_odrive_control" type="system">
             <hardware>

Commit message: add transmission

File: src/rove_description/urdf/rove.ros2_control.urdf.xacro (robot description, xacro)
@@ -46,4 +46,36 @@
                 <state_interface name="effort"/>
             </joint>
+            <transmission name="transmission_fr">
+                <plugin>transmission_interface/SimpleTransmission</plugin>
+                <actuator name="actuator_fr" role="actuator_fr"/>
+                <joint name="track_fr_j" role="track_fr_j">
+                  <mechanical_reduction>30.76923077</mechanical_reduction>
+                  <offset>0.0</offset>
+                </joint>
+              </transmission>
+              <transmission name="transmission_rr">
+                <plugin>transmission_interface/SimpleTransmission</plugin>
+                <actuator name="actuator_rr" role="actuator_rr"/>
+                <joint name="track_rr_j" role="track_rr_j">
+                  <mechanical_reduction>30.76923077</mechanical_reduction>
+                  <offset>0.0</offset>
+                </joint>
+              </transmission>
+              <transmission name="transmission_fl">
+                <plugin>transmission_interface/SimpleTransmission</plugin>
+                <actuator name="actuator_fl" role="actuator_fl"/>
+                <joint name="track_fl_j" role="track_fl_j">
+                  <mechanical_reduction>30.76923077</mechanical_reduction>
+                  <offset>0.0</offset>
+                </joint>
+              </transmission>
+              <transmission name="transmission_rl">
+                <plugin>transmission_interface/SimpleTransmission</plugin>
+                <actuator name="actuator_rl" role="actuator_rl"/>
+                <joint name="track_rl_j" role="track_rl_j">
+                  <mechanical_reduction>30.76923077</mechanical_reduction>
+                  <offset>0.0</offset>
+                </joint>
+              </transmission>
             <!-- <joint name="track_rl_j">
                 <param name="node_id">1</param>

Commit message: arrange mapping

File: src/rove_description/urdf/rove.ros2_control.urdf.xacro (robot description, xacro)
@@ -1,5 +1,4 @@
 <?xml version="1.0"?>
 <robot xmlns:xacro="http://www.ros.org/wiki/xacro">
-    <xacro:include filename="$(find rove_tracks)/urdf/rove_track.urdf.xacro"/>
     <xacro:macro name="rove_odrive_motor" params="position suffix id">
         <xacro:unless value="${(id == -1)}">
@@ -46,36 +45,4 @@
                 <state_interface name="effort"/>
             </joint>
-            <transmission name="transmission_fr">
-                <plugin>transmission_interface/SimpleTransmission</plugin>
-                <actuator name="actuator_fr" role="actuator_fr"/>
-                <joint name="track_fr_j" role="track_fr_j">
-                  <mechanical_reduction>30.76923077</mechanical_reduction>
-                  <offset>0.0</offset>
-                </joint>
-              </transmission>
-              <transmission name="transmission_rr">
-                <plugin>transmission_interface/SimpleTransmission</plugin>
-                <actuator name="actuator_rr" role="actuator_rr"/>
-                <joint name="track_rr_j" role="track_rr_j">
-                  <mechanical_reduction>30.76923077</mechanical_reduction>
-                  <offset>0.0</offset>
-                </joint>
-              </transmission>
-              <transmission name="transmission_fl">
-                <plugin>transmission_interface/SimpleTransmission</plugin>
-                <actuator name="actuator_fl" role="actuator_fl"/>
-                <joint name="track_fl_j" role="track_fl_j">
-                  <mechanical_reduction>30.76923077</mechanical_reduction>
-                  <offset>0.0</offset>
-                </joint>
-              </transmission>
-              <transmission name="transmission_rl">
-                <plugin>transmission_interface/SimpleTransmission</plugin>
-                <actuator name="actuator_rl" role="actuator_rl"/>
-                <joint name="track_rl_j" role="track_rl_j">
-                  <mechanical_reduction>30.76923077</mechanical_reduction>
-                  <offset>0.0</offset>
-                </joint>
-              </transmission>
             <!-- <joint name="track_rl_j">
                 <param name="node_id">1</param>
@@ -132,6 +99,4 @@
     <xacro:macro name="rove_ros2_control">
         <xacro:odrive_control/>
-        <!-- <xacro:track_control suffix="l"/> -->
-        <!-- <xacro:track_control suffix="r"/> -->
     </xacro:macro>
 </robot>

Commit message: Cleaned up ros2 control xacro, added macros, fixed cmd_vel for diffdrive

File: src/rove_description/urdf/rove.ros2_control.urdf.xacro (robot description, xacro)
@@ -1,12 +1,29 @@
 <?xml version="1.0"?>
 <robot xmlns:xacro="http://www.ros.org/wiki/xacro">
-    <xacro:macro name="rove_odrive_motor" params="position suffix id">
+    <xacro:macro name="track_motor_control" params="suffix nodeid">
+        <joint name="track_${suffix}_j">
+            <param name="node_id">${nodeid}</param>
+            <command_interface name="velocity"/>
+            <state_interface name="position"/>
+            <state_interface name="velocity"/>
+            <state_interface name="effort"/>
+        </joint>
+    </xacro:macro>
+    <xacro:macro name="track_fake_motor_control" params="suffix">
+        <joint name="track_${suffix}_j">
+            <command_interface name="velocity"/>
+            <state_interface name="position"/>
+            <state_interface name="velocity"/>
+            <state_interface name="effort"/>
+        </joint>
+    </xacro:macro>
+    <xacro:macro name="rove_odrive_motor" params="suffix id">
         <xacro:unless value="${(id == -1)}">
-            <xacro:track_motor_control position="${position}" suffix="${suffix}" nodeid="${id}"/>
+            <xacro:track_motor_control suffix="${suffix}" nodeid="${id}"/>
         </xacro:unless>
     </xacro:macro>
-    <xacro:macro name="rove_fake_odrive_motor" params="position suffix id">
+    <xacro:macro name="rove_fake_odrive_motor" params="suffix id">
         <xacro:if value="${(id == -1)}">
-            <xacro:track_fake_motor_control position="${position}" suffix="${suffix}"/>
+            <xacro:track_fake_motor_control suffix="${suffix}"/>
         </xacro:if>
     </xacro:macro>
@@ -17,86 +34,18 @@
                 <param name="can">can0</param>
             </hardware>
-            <joint name="track_fr_j">
-                <param name="node_id">23</param>
-                <command_interface name="velocity"/>
-                <state_interface name="position"/>
-                <state_interface name="velocity"/>
-                <state_interface name="effort"/>
-            </joint>
-            <joint name="track_rr_j">
-                <param name="node_id">24</param>
-                <command_interface name="velocity"/>
-                <state_interface name="position"/>
-                <state_interface name="velocity"/>
-                <state_interface name="effort"/>
-            </joint>
-            <joint name="track_fl_j">
-                <param name="node_id">21</param>
-                <command_interface name="velocity"/>
-                <state_interface name="position"/>
-                <state_interface name="velocity"/>
-                <state_interface name="effort"/>
-            </joint>
-            <joint name="track_rl_j">
-                <param name="node_id">22</param>
-                <command_interface name="velocity"/>
-                <state_interface name="position"/>
-                <state_interface name="velocity"/>
-                <state_interface name="effort"/>
-            </joint>
-            <!-- <joint name="track_rl_j">
-                <param name="node_id">1</param>
-            </joint> -->
-            <!-- <xacro:rove_odrive_motor position="f" suffix="l" id="${fl_id}"/>
-            <xacro:rove_odrive_motor position="r" suffix="l" id="${rl_id}"/>
-            <xacro:rove_odrive_motor position="f" suffix="r" id="${fr_id}"/>
-            <xacro:rove_odrive_motor position="r" suffix="r" id="${rr_id}"/> -->
+            <xacro:rove_odrive_motor suffix="fl" id="${fl_id}"/>
+            <xacro:rove_odrive_motor suffix="rl" id="${rl_id}"/>
+            <xacro:rove_odrive_motor suffix="fr" id="${fr_id}"/>
+            <xacro:rove_odrive_motor suffix="rr" id="${rr_id}"/>
         </ros2_control>
-        <!-- <ros2_control name="fake_odrive_control" type="system">
-            <hardware>
-                <plugin>mock_components/GenericSystem</plugin>
-                <param name="calculate_dynamics">true</param>
-            </hardware>
-            <<joint name="track_fl_j">
-                <param name="node_id">1</param>
-                <command_interface name="velocity"/>
-                <state_interface name="position"/>
-                <state_interface name="velocity"/>
-                <state_interface name="effort"/>
-            </joint>
-            <joint name="track_rl_j">
-                <param name="node_id">2</param>
-                <command_interface name="velocity"/>
-                <state_interface name="position"/>
-                <state_interface name="velocity"/>
-                <state_interface name="effort"/>
-            </joint>
-            <joint name="track_fr_j">
-                <param name="node_id">3</param>
-                <command_interface name="velocity"/>
-                <state_interface name="position"/>
-                <state_interface name="velocity"/>
-                <state_interface name="effort"/>
-            </joint>
-            <joint name="track_rr_j">
-                <param name="node_id">3</param>
-                <command_interface name="velocity"/>
-                <state_interface name="position"/>
-                <state_interface name="velocity"/>
-                <state_interface name="effort"/>
-            </joint>
-        </ros2_control> -->
-        <!-- <ros2_control name="fake_odrive_control" type="system">
+        <ros2_control name="fake_odrive_control" type="system">
             <hardware>
                 <plugin>mock_components/GenericSystem</plugin>
             </hardware>
-            <xacro:rove_fake_odrive_motor position="f" suffix="l" id="${fl_id}"/>
-            <xacro:rove_fake_odrive_motor position="r" suffix="l" id="${rl_id}"/>
-            <xacro:rove_fake_odrive_motor position="f" suffix="r" id="${fr_id}"/>
-            <xacro:rove_fake_odrive_motor position="r" suffix="r" id="${rr_id}"/>
-        </ros2_control> -->
-    </xacro:macro>
-    <xacro:macro name="rove_ros2_control">
-        <xacro:odrive_control/>
+            <xacro:rove_fake_odrive_motor suffix="fl" id="${fl_id}"/>
+            <xacro:rove_fake_odrive_motor suffix="rl" id="${rl_id}"/>
+            <xacro:rove_fake_odrive_motor suffix="fr" id="${fr_id}"/>
+            <xacro:rove_fake_odrive_motor suffix="rr" id="${rr_id}"/>
+        </ros2_control>
     </xacro:macro>
 </robot>

File: src/rove_description/urdf/rove.urdf.xacro (robot description, xacro)
@@ -37,5 +37,5 @@
     </link>
     <!-- <xacro:rove_ros2_control/> -->
-    <xacro:odrive_control fl_id="0" rl_id="-1" fr_id="-1" rr_id="-1"/>
+    <xacro:odrive_control fl_id="21" rl_id="22" fr_id="23" rr_id="24"/>
     <!-- Insert ovis on top of rove -->
     <!-- <xacro:property name="robot_root" value="base_link" />

Commit message: Adding flippers

File: src/rove_description/urdf/rove.ros2_control.urdf.xacro (robot description, xacro)
@@ -22,4 +22,25 @@
         </joint>
     </xacro:macro>
+    <xacro:macro name="flipper_motor_control" params="suffix nodeid">
+        <joint name="flipper_${suffix}_j">
+            <param name="node_id">${nodeid}</param>
+            <command_interface name="position"/>
+            <state_interface name="position"/>
+            <state_interface name="velocity"/>
+            <state_interface name="effort"/>
+            <state_interface name="voltage"/>
+            <state_interface name="current"/>
+        </joint>
+    </xacro:macro>
+    <xacro:macro name="flipper_fake_motor_control" params="suffix">
+        <joint name="flipper_${suffix}_j">
+            <command_interface name="position"/>
+            <state_interface name="position"/>
+            <state_interface name="velocity"/>
+            <state_interface name="effort"/>
+            <state_interface name="voltage"/>
+            <state_interface name="current"/>
+        </joint>
+    </xacro:macro>
     <xacro:macro name="rove_odrive_motor" params="suffix id">
         <xacro:unless value="${(id == -1)}">
@@ -32,5 +53,15 @@
         </xacro:if>
     </xacro:macro>
-    <xacro:macro name="odrive_control" params="fl_id:=21 rl_id:=22 fr_id:=23 rr_id:=24">
+    <xacro:macro name="rove_odrive_flipper" params="suffix id">
+        <xacro:unless value="${(id == -1)}">
+            <xacro:flipper_motor_control suffix="${suffix}" nodeid="${id}"/>
+        </xacro:unless>
+    </xacro:macro>
+    <xacro:macro name="rove_fake_odrive_flipper" params="suffix id">
+        <xacro:if value="${(id == -1)}">
+            <xacro:flipper_fake_motor_control suffix="${suffix}"/>
+        </xacro:if>
+    </xacro:macro>
+    <xacro:macro name="odrive_control" params="fl_id:=21 rl_id:=22 fr_id:=23 rr_id:=24 ffl_id:=11 frl_id:=12 ffr_id:=13 frr_id:=14">
         <ros2_control name="odrive_control" type="system">
             <hardware>
@@ -42,4 +73,8 @@
             <xacro:rove_odrive_motor suffix="fr" id="${fr_id}"/>
             <xacro:rove_odrive_motor suffix="rr" id="${rr_id}"/>
+            <xacro:rove_odrive_motor suffix="fl" id="${ffl_id}"/>
+            <xacro:rove_odrive_motor suffix="rl" id="${frl_id}"/>
+            <xacro:rove_odrive_motor suffix="fr" id="${ffr_id}"/>
+            <xacro:rove_odrive_motor suffix="rr" id="${frr_id}"/>
         </ros2_control>
         <ros2_control name="fake_odrive_control" type="system">
@@ -51,4 +86,8 @@
             <xacro:rove_fake_odrive_motor suffix="fr" id="${fr_id}"/>
             <xacro:rove_fake_odrive_motor suffix="rr" id="${rr_id}"/>
+            <xacro:rove_fake_odrive_flipper suffix="fl" id="${ffl_id}"/>
+            <xacro:rove_fake_odrive_flipper suffix="rl" id="${frl_id}"/>
+            <xacro:rove_fake_odrive_flipper suffix="fr" id="${ffr_id}"/>
+            <xacro:rove_fake_odrive_flipper suffix="rr" id="${frr_id}"/>
         </ros2_control>
     </xacro:macro>
