Commit message: test for flipper gazebo

File: src/rove_description/urdf/flipper.urdf.xacro (robot description, xacro)
@@ -10,4 +10,10 @@
             <xacro:property name="joint_origin" value="${flipper_j_x} ${-flipper_j_y} ${flipper_j_z}"/>
             <xacro:property name="joint_axis" value="0 -1 0"/>
+            <xacro:property name="node_id" value="13"/>
+            <command_interface name="position">
+                <param name="min">-1</param>
+                <param name="max">1</param>
+            </command_interface>
+            <state_interface name="position"/>
         </xacro:if>
         <xacro:if value="${(suffix == 'fl')}">
@@ -15,4 +21,10 @@
             <xacro:property name="joint_origin" value="${flipper_j_x} ${flipper_j_y}  ${flipper_j_z}"/>
             <xacro:property name="joint_axis" value="0 -1 0"/>
+            <xacro:property name="node_id" value="11"/>
+            <command_interface name="position">
+                <param name="min">-1</param>
+                <param name="max">1</param>
+            </command_interface>
+            <state_interface name="position"/>
         </xacro:if>
         <xacro:if value="${(suffix == 'rr')}">
@@ -20,4 +32,5 @@
             <xacro:property name="joint_origin" value="${-flipper_j_x} ${-flipper_j_y}  ${flipper_j_z}"/>
             <xacro:property name="joint_axis" value="0 1 0"/>
+            <xacro:property name="node_id" value="11"/>
         </xacro:if>
         <xacro:if value="${(suffix == 'rl')}">
@@ -25,4 +38,5 @@
             <xacro:property name="joint_origin" value="${-flipper_j_x} ${flipper_j_y} ${flipper_j_z}"/>
             <xacro:property name="joint_axis" value="0 1 0"/>
+            <xacro:property name="node_id" value="11"/>
         </xacro:if>
         <joint name="flipper_${suffix}_j" type="continuous">

Commit message: merge 3d lidar + 3d cam

File: src/rove_description/urdf/flipper.urdf.xacro (robot description, xacro)
@@ -7,46 +7,50 @@
         <xacro:property name="flipper_j_z" value="0.0889" />
         <xacro:if value="${(suffix == 'fr')}">
-            <xacro:property name="mesh_rotation" value="0 0 ${pi}"/>
-            <xacro:property name="joint_origin" value="${flipper_j_x} ${-flipper_j_y} ${flipper_j_z}"/>
-            <xacro:property name="joint_axis" value="0 -1 0"/>
+            <xacro:property name="mesh_rotation" value="0 0 ${pi}" />
+            <xacro:property name="joint_origin"
+                value="${flipper_j_x} ${-flipper_j_y} ${flipper_j_z}" />
+            <xacro:property name="joint_axis" value="0 -1 0" />
         </xacro:if>
         <xacro:if value="${(suffix == 'fl')}">
             <xacro:property name="mesh_rotation" value="0 ${pi} 0" />
-            <xacro:property name="joint_origin" value="${flipper_j_x} ${flipper_j_y}  ${flipper_j_z}"/>
-            <xacro:property name="joint_axis" value="0 -1 0"/>
+            <xacro:property name="joint_origin"
+                value="${flipper_j_x} ${flipper_j_y}  ${flipper_j_z}" />
+            <xacro:property name="joint_axis" value="0 -1 0" />
         </xacro:if>
         <xacro:if value="${(suffix == 'rr')}">
             <xacro:property name="mesh_rotation" value="${pi} 0 0" />
-            <xacro:property name="joint_origin" value="${-flipper_j_x} ${-flipper_j_y}  ${flipper_j_z}"/>
-            <xacro:property name="joint_axis" value="0 1 0"/>
+            <xacro:property name="joint_origin"
+                value="${-flipper_j_x} ${-flipper_j_y}  ${flipper_j_z}" />
+            <xacro:property name="joint_axis" value="0 1 0" />
         </xacro:if>
         <xacro:if value="${(suffix == 'rl')}">
             <xacro:property name="mesh_rotation" value="0 0 0" />
-            <xacro:property name="joint_origin" value="${-flipper_j_x} ${flipper_j_y} ${flipper_j_z}"/>
-            <xacro:property name="joint_axis" value="0 1 0"/>
+            <xacro:property name="joint_origin"
+                value="${-flipper_j_x} ${flipper_j_y} ${flipper_j_z}" />
+            <xacro:property name="joint_axis" value="0 1 0" />
         </xacro:if>
         <joint name="flipper_${suffix}_j" type="continuous">
-            <origin xyz="${joint_origin}" rpy="0 0 0"/>
-            <axis xyz="${joint_axis}"/>
-            <parent link="base_link"/>
-            <child link="flipper_${suffix}"/>
-            <limit effort="10.0" velocity="0.5"/>
-            <dynamics damping="50.0" friction="50"/>
+            <origin xyz="${joint_origin}" rpy="0 0 0" />
+            <axis xyz="${joint_axis}" />
+            <parent link="base_link" />
+            <child link="flipper_${suffix}" />
+            <limit effort="10.0" velocity="0.5" />
+            <dynamics damping="50.0" friction="50" />
         </joint>
         <link name="flipper_${suffix}">
             <visual>
-                <origin xyz="0 0 0" rpy="${mesh_rotation}"/>
+                <origin xyz="0 0 0" rpy="${mesh_rotation}" />
                 <geometry>
-                    <mesh filename="file://$(find rove_description)/meshes/flipper.stl"/>
+                    <mesh filename="file://$(find rove_description)/meshes/flipper.stl" />
                 </geometry>
-                <material name="rubber_color"/>
+                <material name="rubber_color" />
             </visual>
             <collision>
-                <origin xyz="0 0 0" rpy="${mesh_rotation}"/>
+                <origin xyz="0 0 0" rpy="${mesh_rotation}" />
                 <geometry>
-                    <mesh filename="file://$(find rove_description)/meshes/flipper.stl"/>
+                    <mesh filename="file://$(find rove_description)/meshes/flipper.stl" />
                 </geometry>
                 <surface>
-<friction>
+                    <friction>
                         <ode>
                             <mu>0.65</mu>
@@ -55,5 +59,5 @@
                     </friction>
                     <contact>
-                        <ode/>
+                        <ode />
                     </contact>
                 </surface>
@@ -62,21 +66,22 @@
             <!-- TODO PUT ACTUAL INERTIAL VALUES I DON'T KNOW WHAT THIS REPRESENTS NOW -->
             <inertial>
-                <origin xyz="0 0 0.5" rpy="0 0 0"/>
-                <mass value="1"/>
-                <inertia ixx="100"  ixy="0"  ixz="0" iyy="100" iyz="0" izz="100" />
+                <origin xyz="0 0 0.5" rpy="0 0 0" />
+                <mass value="1" />
+                <inertia ixx="0" ixy="0" ixz="0" iyy="0" iyz="0" izz="0" />
             </inertial>
         </link>
         <gazebo>
-            <plugin name='gz::sim::systems::TrackController' filename='gz-sim-track-controller-system'>
-                    <link>flipper_${suffix}</link>
-                    <min_velocity>-3.0</min_velocity>
-                    <max_velocity>3.0</max_velocity>
-                    <!--debug>1</debug-->
+            <plugin name='gz::sim::systems::TrackController'
+                filename='gz-sim-track-controller-system'>
+                <link>flipper_${suffix}</link>
+                <min_velocity>-3.0</min_velocity>
+                <max_velocity>3.0</max_velocity>
+                <!--debug>1</debug-->
             </plugin>
         </gazebo>
     </xacro:macro>
-    <xacro:flipper suffix="fr"/>
-    <xacro:flipper suffix="fl"/>
-    <xacro:flipper suffix="rr"/>
-    <xacro:flipper suffix="rl"/>
+    <xacro:flipper suffix="fr" />
+    <xacro:flipper suffix="fl" />
+    <xacro:flipper suffix="rr" />
+    <xacro:flipper suffix="rl" />
 </robot>

File: src/rove_description/urdf/rove.urdf.xacro (robot description, xacro)
@@ -33,5 +33,5 @@
             <origin xyz="0 0 0.5" rpy="0 0 0"/>
             <mass value="80"/>
-            <inertia ixx="100"  ixy="0"  ixz="0" iyy="100" iyz="0" izz="100" />
+            <inertia ixx="1"  ixy="0"  ixz="0" iyy="1" iyz="0" izz="1" />
         </inertial>
     </link>

File: src/rove_description/urdf/sensor.urdf.xacro (robot description, xacro)
@@ -11,14 +11,12 @@
         <parent link="sensor_link" />
         <child link="camera_link" />
-        <origin xyz="0.1 0 0.4" rpy="-1.57 0 -1.57" />
+        <origin xyz="0.1 0 0" rpy="-1.57 0 -1.57" />
     </joint>
     <link name="camera_link">
         <inertial>
-            <origin xyz="0 0 0" rpy="0 0 0" />
             <mass value="0.1" />
             <inertia ixx="0.0001" ixy="0.0" ixz="0.0" iyy="0.0001" iyz="0.0" izz="0.0001" />
         </inertial>
         <visual>
-            <origin xyz="0 0 0" rpy="0 0 0" />
             <geometry>
                 <cylinder length="0.1" radius="0.1" />
@@ -75,6 +73,6 @@
                 <horizontal_fov>1.88</horizontal_fov>
                 <image>
-                    <width>256</width>
-                    <height>256</height>
+                    <width>1344</width>
+                    <height>376</height>
                     <format>R_FLOAT32</format>
                 </image>
@@ -94,6 +92,6 @@
                 <horizontal_fov>1.88</horizontal_fov>
                 <image>
-                    <width>256</width>
-                    <height>256</height>
+                    <width>1344</width>
+                    <height>376</height>
                     <format>R_FLOAT32</format>
                 </image>

File: src/rove_description/urdf/track.urdf.xacro (robot description, xacro)
@@ -57,5 +57,5 @@
                 <origin xyz="0 0 0" rpy="0 0 0"/>
                 <mass value="1"/>
-                <inertia ixx="100"  ixy="0"  ixz="0" iyy="100" iyz="0" izz="100" />
+                <inertia ixx="0"  ixy="0"  ixz="0" iyy="0" iyz="0" izz="0" />
             </inertial>
         </link>

Commit message: add flipper url link

File: src/rove_description/urdf/flipper.urdf.xacro (robot description, xacro)
@@ -39,4 +39,11 @@
         </joint>
         <link name="flipper_${suffix}">
+            <visual>
+                <origin xyz="0 0 0" rpy="${mesh_rotation}" />
+                <geometry>
+                    <mesh filename="https://raw.githubusercontent.com/clubcapra/rove/main/src/rove_description/meshes/flipper.stl"/>
+                </geometry>
+                <material name="rubber_color" />
+            </visual>
             <visual>
                 <origin xyz="0 0 0" rpy="${mesh_rotation}" />

File: src/rove_description/urdf/rove.urdf.xacro (robot description, xacro)
@@ -20,4 +20,11 @@
             <origin xyz="0 0 0" rpy="0 0 0"/>
             <geometry>
+                <mesh filename="https://raw.githubusercontent.com/clubcapra/rove/main/src/rove_description/meshes/base.stl"/>
+            </geometry>
+            <material name="frame_color"/>
+        </visual>
+        <visual>
+            <origin xyz="0 0 0" rpy="0 0 0"/>
+            <geometry>
                 <mesh filename="file://$(find rove_description)/meshes/base.stl"/>
             </geometry>
@@ -38,6 +45,6 @@
     <!-- <xacro:rove_ros2_control/> -->
      <!-- Put these at -1 to mock the motors if working without the motors -->
+    <!-- <xacro:odrive_control fl_id="21" rl_id="22" fr_id="23" rr_id="24"/> -->
     <xacro:odrive_control fl_id="21" rl_id="22" fr_id="23" rr_id="24"/>
-    <!-- <xacro:odrive_control fl_id="-1" rl_id="-1" fr_id="-1" rr_id="-1"/> -->
     <!-- Insert ovis on top of rove -->
     <!-- <xacro:property name="robot_root" value="base_link" />

File: src/rove_description/urdf/track.urdf.xacro (robot description, xacro)
@@ -28,4 +28,11 @@
         </joint>
         <link name="track_${suffix}">
+            <visual>
+                <origin xyz="0 0 0"/>
+                <geometry>
+                    <mesh filename="https://raw.githubusercontent.com/clubcapra/rove/main/src/rove_description/meshes/track.stl"/>
+                </geometry>
+                <material name="rubber_color" />
+            </visual>
             <visual>
                 <origin xyz="0 0 0" rpy="0 0 0"/>

Commit message: Fixed sim

File: src/rove_description/urdf/flipper.urdf.xacro (robot description, xacro)
@@ -39,11 +39,4 @@
         </joint>
         <link name="flipper_${suffix}">
-            <visual>
-                <origin xyz="0 0 0" rpy="${mesh_rotation}" />
-                <geometry>
-                    <mesh filename="https://raw.githubusercontent.com/clubcapra/rove/main/src/rove_description/meshes/flipper.stl"/>
-                </geometry>
-                <material name="rubber_color" />
-            </visual>
             <visual>
                 <origin xyz="0 0 0" rpy="${mesh_rotation}" />

File: src/rove_description/urdf/rove.urdf.xacro (robot description, xacro)
@@ -16,13 +16,11 @@
     <xacro:include filename="$(find rove_description)/urdf/rove.ros2_control.urdf.xacro" />
     <!-- <xacro:include filename="$(find ovis_description)/urdf/ovis.urdf.xacro" /> -->
+    <!-- Workaround for KDL not allowing root link to have inertia -->
+    <!-- <link name="dummy_root"/>
+    <joint name="fixed_base" type="fixed">
+        <parent link="dummy_root"/>
+        <child link="base_link"/>
+    </joint> -->
     <link name="base_link">
-        <visual>
-            <origin xyz="0 0 0" rpy="0 0 0" />
-            <geometry>
-                <mesh
-                    filename="https://raw.githubusercontent.com/clubcapra/rove/main/src/rove_description/meshes/base.stl" />
-            </geometry>
-            <material name="frame_color" />
-        </visual>
         <visual>
             <origin xyz="0 0 0" rpy="0 0 0" />

File: src/rove_description/urdf/track.urdf.xacro (robot description, xacro)
@@ -28,11 +28,4 @@
         </joint>
         <link name="track_${suffix}">
-            <visual>
-                <origin xyz="0 0 0"/>
-                <geometry>
-                    <mesh filename="https://raw.githubusercontent.com/clubcapra/rove/main/src/rove_description/meshes/track.stl"/>
-                </geometry>
-                <material name="rubber_color" />
-            </visual>
             <visual>
                 <origin xyz="0 0 0" rpy="0 0 0"/>
