Commit message: add basic navigation

File: src/rove_description/urdf/gazebo.urdf.xacro (robot description, xacro)
@@ -1,22 +1,9 @@
 <?xml version="1.0"?>
 <robot xmlns:xacro="http://www.ros.org/wiki/xacro">
-    <gazebo reference="imu_link">
-        <sensor name="imu_sensor" type="imu">
-            <gz_frame_id>rove/imu_link</gz_frame_id>
-            <update_rate>50</update_rate>
-            <visualize>false</visualize>
-            <topic>imu</topic>
-            <always_on>false</always_on>
-        </sensor>
-    </gazebo>
-    <link name="imu_link" />
-    <joint name="imu_link_joint" type="fixed">
-        <parent link="base_link"/>
-        <child link="imu_link"/>
-    </joint>
     <gazebo>
         <plugin
             filename="ignition-gazebo-joint-state-publisher-system"
             name="ignition::gazebo::systems::JointStatePublisher">
+            <topic>joint_states</topic>
         </plugin>
         <plugin
@@ -24,5 +11,5 @@
             name="ignition::gazebo::systems::Imu">
         </plugin>
-        <plugin name="gz::sim::systems::TrackedVehicle" filename="ignition-gazebo-tracked-vehicle-system">
+        <plugin name="gz::sim::systems::TrackedVehicle" filename="gz-sim-tracked-vehicle-system">
             <left_track><link>track_l</link></left_track>
             <left_track><link>flipper_fl</link></left_track>
@@ -34,6 +21,11 @@
             <tracks_separation>0.4</tracks_separation>
             <tracks_height>0.18094</tracks_height>
-            <steering_efficiency>0.5</steering_efficiency>
-            <child_frame_id>rove/base_link</child_frame_id>
+            <steering_efficiency>1</steering_efficiency>
+             <topic>cmd_vel</topic>
+            <odom_topic>odom</odom_topic>
+            <frame_id>odom</frame_id>
+            <child_frame_id>base_link</child_frame_id>
+            <odom_publisher_frequency>30</odom_publisher_frequency>
+            <tf_topic>/tf</tf_topic>
         </plugin>
         <plugin

File: src/rove_description/urdf/lidar.urdf.xacro (robot description, xacro)
@@ -4,8 +4,8 @@
     <joint name="laser_joint" type="fixed">
         <parent link="base_link"/>
-        <child link="laser_frame"/>
-        <origin xyz="0.0 0 0.4" rpy="0 0 0"/>
+        <child link="base_scan"/>
+      <origin xyz="0.0 0 0.4" rpy="0 0 0"/>
     </joint>
-    <link name="laser_frame">
+    <link name="base_scan">
         <visual>
             <geometry>
@@ -26,12 +26,13 @@
         </inertial>
     </link>
-    <gazebo reference="laser_frame">
+    <gazebo reference="base_scan">
         <material>Gazebo/Black</material>
         <sensor name='laser_sensor_frame' type='gpu_lidar'>
-            <gz_frame_id>rove/laser_frame</gz_frame_id>
             <pose> 0 0 0 0 0 0 </pose>
-            <visualize>false</visualize>
-            <always_on>false</always_on>
-            <update_rate>10</update_rate>
+            <visualize>true</visualize>
+            <always_on>true</always_on>
+            <update_rate>5</update_rate>
+            <topic>scan</topic>
+            <gz_frame_id>base_scan</gz_frame_id>
             <ray>
                 <scan>

Commit message: add base footprint + fix odom

File: src/rove_description/urdf/gazebo.urdf.xacro (robot description, xacro)
@@ -19,5 +19,5 @@
             <right_track><link>flipper_rr</link></right_track>
              <!-- TODO PUT ACTUAL VALUES -->
-            <tracks_separation>0.4</tracks_separation>
+            <tracks_separation>0.63</tracks_separation>
             <tracks_height>0.18094</tracks_height>
             <steering_efficiency>1</steering_efficiency>
@@ -25,5 +25,5 @@
             <odom_topic>odom</odom_topic>
             <frame_id>odom</frame_id>
-            <child_frame_id>base_link</child_frame_id>
+            <child_frame_id>base_footprint</child_frame_id>
             <odom_publisher_frequency>30</odom_publisher_frequency>
             <tf_topic>/tf</tf_topic>

File: src/rove_description/urdf/rove.urdf.xacro (robot description, xacro)
@@ -14,4 +14,5 @@
     <xacro:include filename="$(find rove_description)/urdf/flipper.urdf.xacro" />
     <xacro:include filename="$(find rove_description)/urdf/track.urdf.xacro" />
+    <link name="base_footprint"/>
     <link name="base_link">
         <visual>
@@ -34,3 +35,8 @@
         </inertial>
     </link>
+    <joint name="base_joint" type="fixed">
+        <origin rpy="0 0 0" xyz="0 0 0"/>
+        <parent link="base_footprint"/>
+        <child link="base_link"/>
+    </joint>
 </robot>

Commit message: add better fusion with imu

File: src/rove_description/urdf/gazebo.urdf.xacro (robot description, xacro)
@@ -25,5 +25,4 @@
             <odom_topic>odom</odom_topic>
             <frame_id>odom</frame_id>
-            <child_frame_id>base_footprint</child_frame_id>
             <odom_publisher_frequency>30</odom_publisher_frequency>
             <publish_odom_tf>false</publish_odom_tf>

File: src/rove_description/urdf/rove.urdf.xacro (robot description, xacro)
@@ -16,5 +16,4 @@
     <xacro:include filename="$(find rove_description)/urdf/track.urdf.xacro" />
     <xacro:include filename="$(find ovis_description)/urdf/ovis.urdf.xacro" />
-    <link name="base_footprint"/>
     <link name="base_link">
         <visual>
@@ -37,9 +36,4 @@
         </inertial>
     </link>
-    <joint name="base_joint" type="fixed">
-        <origin rpy="0 0 0" xyz="0 0 0"/>
-        <parent link="base_footprint"/>
-        <child link="base_link"/>
-    </joint>
     <!-- Insert ovis on top of rove -->
     <xacro:property name="robot_root" value="base_link" />

File: src/rove_description/urdf/sensor.urdf.xacro (robot description, xacro)
@@ -28,21 +28,8 @@
         <material>Gazebo/Black</material>
         <sensor name="imu_sensor" type="imu">
-            <gz_frame_id>imu_link</gz_frame_id>
+            <gz_frame_id>sensor_link</gz_frame_id>
             <always_on>true</always_on>
-            <update_rate>200</update_rate>
+            <update_rate>50</update_rate>
             <topic>imu</topic>
-            <imu>
-                <noise>
-                    <type>gaussian</type>
-                    <rate>
-                        <mean>0.0</mean>
-                        <stddev>0.01</stddev>
-                    </rate>
-                    <accel>
-                        <mean>0.0</mean>
-                        <stddev>0.01</stddev>
-                    </accel>
-                </noise>
-            </imu>
         </sensor>
         <sensor name="gps_sensor" type="navsat">

File: src/rove_description/urdf/track.urdf.xacro (robot description, xacro)
@@ -33,6 +33,6 @@
                     <friction>
                         <ode>
-                            <mu>0.65</mu>
-                            <mu2>0.85</mu2>
+                            <mu>1</mu>
+                            <mu2>1</mu2>
                         </ode>
                     </friction>
@@ -51,5 +51,5 @@
         </link>
         <gazebo>
-            <plugin name='gz::sim::systems::TrackController' filename='libignition-gazebo-track-controller-system.so'>
+            <plugin name='gz::sim::systems::TrackController' filename='gz-sim-track-controller-system'>
                     <link>track_${suffix}</link>
                     <min_velocity>-3.0</min_velocity>

File: src/rove_description/urdf/velodyne.urdf.xacro (robot description, xacro)
@@ -60,8 +60,7 @@
     <gazebo reference="${name}_laser">
       <sensor name="${name}" type="gpu_lidar">
-        <update_rate>${update_rate}</update_rate>
         <visualize>true</visualize>
         <always_on>true</always_on>
-        <update_rate>5</update_rate>
+        <update_rate>50</update_rate>
         <topic>scan</topic>
         <gz_frame_id>${name}_laser</gz_frame_id>

Commit message: edit

File: src/rove_description/urdf/gazebo.urdf.xacro (robot description, xacro)
@@ -1,4 +1,5 @@
 <?xml version="1.0"?>
-<robot xmlns:xacro="http://www.ros.org/wiki/xacro">
+<robot xmlns:xacro="http://www.ros.org/wiki/xacro"
+    name="rove">
     <gazebo>
         <plugin

File: src/rove_description/urdf/track.urdf.xacro (robot description, xacro)
@@ -1,4 +1,4 @@
 <?xml version="1.0"?>
-<robot xmlns:xacro="http://www.ros.org/wiki/xacro">
+<robot xmlns:xacro="http://www.ros.org/wiki/xacro" name="track">
     <!--Track xacro-->
     <xacro:macro name="track" params="suffix">
@@ -63,4 +63,6 @@
             <inertial>
                 <origin xyz="0 0 0" rpy="0 0 0"/>
+                <mass value="0"/>
+                <inertia ixx="100"  ixy="0"  ixz="0" iyy="0" iyz="0" izz="100"/>
             </inertial>
         </link>
@@ -68,4 +70,6 @@
             <inertial>
                 <origin xyz="0 0 0" rpy="0 0 0"/>
+                <mass value="0"/>
+                <inertia ixx="100"  ixy="0"  ixz="0" iyy="0" iyz="0" izz="100"/>
             </inertial>
         </link>

Commit message: it works ! long live the friction

File: src/rove_description/urdf/gazebo.urdf.xacro (robot description, xacro)
@@ -34,4 +34,11 @@
         </plugin>
         <plugin filename="gz-sim-navsat-system" name="gz::sim::systems::NavSat"/>
+        <gazebo reference="friction_plate_base">
+            <material>Gazebo/Grey</material>
+            <mu1>100.0</mu1>
+            <mu2>100.0</mu2>
+            <kp>1000000.0</kp>
+            <kd>1.0</kd>
+        </gazebo>
     </gazebo>
 </robot>

File: src/rove_description/urdf/rove.urdf.xacro (robot description, xacro)
@@ -2,11 +2,11 @@
 <robot name="rove" xmlns:xacro="http://www.ros.org/wiki/xacro">
     <material name="rubber_color">
-        <color rgba="0.1 0.1 0.1 1.0"/>
+        <color rgba="0.1 0.1 0.1 1.0" />
     </material>
     <material name="frame_color">
-        <color rgba="0.5 0.5 0.5 1.0"/>
+        <color rgba="0.5 0.5 0.5 1.0" />
     </material>
     <material name="lidar_color">
-        <color rgba="1 0 0 1.0"/>
+        <color rgba="1 0 0 1.0" />
     </material>
     <xacro:include filename="$(find rove_description)/urdf/gazebo.urdf.xacro" />
@@ -18,38 +18,116 @@
     <link name="base_link">
         <visual>
-            <origin xyz="0 0 0" rpy="0 0 0"/>
+            <origin xyz="0 0 0" rpy="0 0 0" />
             <geometry>
-                <mesh filename="https://raw.githubusercontent.com/clubcapra/rove/main/src/rove_description/meshes/base.stl"/>
+                <mesh
+                    filename="https://raw.githubusercontent.com/clubcapra/rove/main/src/rove_description/meshes/base.stl" />
             </geometry>
-            <material name="frame_color"/>
+            <material name="frame_color" />
         </visual>
         <visual>
-            <origin xyz="0 0 0" rpy="0 0 0"/>
+            <origin xyz="0 0 0" rpy="0 0 0" />
             <geometry>
-                <mesh filename="file://$(find rove_description)/meshes/base.stl"/>
+                <mesh filename="file://$(find rove_description)/meshes/base.stl" />
             </geometry>
-            <material name="frame_color"/>
+            <material name="frame_color" />
         </visual>
         <collision>
-            <origin xyz="0 0 0" rpy="0 0 0"/>
+            <origin xyz="0 0 0" rpy="0 0 0" />
             <geometry>
-                <mesh filename="file://$(find rove_description)/meshes/base.stl"/>
+                <mesh filename="file://$(find rove_description)/meshes/base.stl" />
             </geometry>
         </collision>
         <inertial>
-            <origin xyz="0 0 0.5" rpy="0 0 0"/>
-            <mass value="80"/>
-            <inertia ixx="1"  ixy="0"  ixz="0" iyy="1" iyz="0" izz="1" />
+            <origin xyz="0 0 0.5" rpy="0 0 0" />
+            <mass value="80" />
+            <inertia ixx="1" ixy="0" ixz="0" iyy="1" iyz="0" izz="1" />
         </inertial>
     </link>
+    <link name="friction_plate_base">
+        <visual>
+            <origin xyz="0 0 0" rpy="0 0 0" />
+            <geometry>
+                <box size="0.3 0.3 0.01" />
+            </geometry>
+            <material name="frame_color" />
+        </visual>
+        <visual>
+            <origin xyz="0.14 0 0.02" rpy="0 0 0" />
+            <geometry>
+                <box size="0.02 0.3 0.04" />
+            </geometry>
+            <material name="frame_color" />
+        </visual>
+        <visual>
+            <origin xyz="-0.14 0 0.02" rpy="0 0 0" />
+            <geometry>
+                <box size="0.02 0.3 0.04" />
+            </geometry>
+            <material name="frame_color" />
+        </visual>
+        <visual>
+            <origin xyz="0 0.14 0.02" rpy="0 0 0" />
+            <geometry>
+                <box size="0.26 0.02 0.04" />
+            </geometry>
+            <material name="frame_color" />
+        </visual>
+        <visual>
+            <origin xyz="0 -0.14 0.02" rpy="0 0 0" />
+            <geometry>
+                <box size="0.26 0.02 0.04" />
+            </geometry>
+            <material name="frame_color" />
+        </visual>
+        <collision>
+            <origin xyz="0 0 0" rpy="0 0 0" />
+            <geometry>
+                <box size="0.3 0.3 0.01" />
+            </geometry>
+        </collision>
+        <collision>
+            <origin xyz="0.14 0 0.02" rpy="0 0 0" />
+            <geometry>
+                <box size="0.02 0.3 0.04" />
+            </geometry>
+        </collision>
+        <collision>
+            <origin xyz="-0.14 0 0.02" rpy="0 0 0" />
+            <geometry>
+                <box size="0.02 0.3 0.04" />
+            </geometry>
+        </collision>
+        <collision>
+            <origin xyz="0 0.14 0.02" rpy="0 0 0" />
+            <geometry>
+                <box size="0.26 0.02 0.04" />
+            </geometry>
+        </collision>
+        <collision>
+            <origin xyz="0 -0.14 0.02" rpy="0 0 0" />
+            <geometry>
+                <box size="0.26 0.02 0.04" />
+            </geometry>
+        </collision>
+        <inertial>
+            <mass value="1.5" />
+            <inertia ixx="0.02" ixy="0" ixz="0" iyy="0.02" iyz="0" izz="0.02" />
+        </inertial>
+    </link>
+    <joint name="friction_plate_base_joint" type="fixed">
+        <parent link="base_link" />
+        <child link="friction_plate_base" />
+        <origin xyz="0.22 0 0.2" rpy="0 0 0" />
+    </joint>
     <!-- <xacro:rove_ros2_control/> -->
-     <!-- Put these at -1 to mock the motors if working without the motors -->
+    <!-- Put these at -1 to mock the motors if working without the motors -->
     <!-- <xacro:odrive_control fl_id="21" rl_id="22" fr_id="23" rr_id="24"/> -->
     <!-- TODO Fix rr Odrive, it keeps crashing the rest of the drives. IT has been disabled for now. -->
-    <xacro:odrive_control fl_id="21" rl_id="22" fr_id="23" rr_id="24"/>
+    <xacro:odrive_control fl_id="21" rl_id="22" fr_id="23" rr_id="24" />
     <!-- Insert ovis on top of rove -->
     <!-- <xacro:property name="robot_root" value="base_link" />
     <xacro:property name="ovis_robot_namespace" value="rove" />
     <xacro:property name="ovis_base_origin" value="-0.2 0 0.2" />
-    <xacro:ovis base_parent="${robot_root}" prefix="${ovis_robot_namespace}" joint_base_origin_xyz="${ovis_base_origin}" /> -->
+    <xacro:ovis base_parent="${robot_root}" prefix="${ovis_robot_namespace}"
+    joint_base_origin_xyz="${ovis_base_origin}" /> -->
 </robot>

Commit message: add aws small house from to rove

File: src/rove_description/urdf/gazebo.urdf.xacro (robot description, xacro)
@@ -13,10 +13,22 @@
         </plugin>
         <plugin name="gz::sim::systems::TrackedVehicle" filename="gz-sim-tracked-vehicle-system">
-            <left_track><link>track_l</link></left_track>
-            <left_track><link>flipper_fl</link></left_track>
-            <left_track><link>flipper_rl</link></left_track>
-            <right_track><link>track_r</link></right_track>
-            <right_track><link>flipper_fr</link></right_track>
-            <right_track><link>flipper_rr</link></right_track>
+            <left_track>
+                <link>track_l</link>
+            </left_track>
+            <left_track>
+                <link>flipper_fl</link>
+            </left_track>
+            <left_track>
+                <link>flipper_rl</link>
+            </left_track>
+            <right_track>
+                <link>track_r</link>
+            </right_track>
+            <right_track>
+                <link>flipper_fr</link>
+            </right_track>
+            <right_track>
+                <link>flipper_rr</link>
+            </right_track>
             <!-- TODO PUT ACTUAL VALUES -->
             <tracks_separation>0.63</tracks_separation>
@@ -28,10 +40,5 @@
             <child_frame_id>base_link</child_frame_id>
         </plugin>
-        <plugin
-            filename="gz-sim-sensors-system"
-            name="gz::sim::systems::Sensors">
-            <render_engine>ogre2</render_engine>
-        </plugin>
-        <plugin filename="gz-sim-navsat-system" name="gz::sim::systems::NavSat"/>
+        <plugin filename="gz-sim-navsat-system" name="gz::sim::systems::NavSat" />
         <gazebo reference="friction_plate_base">
             <material>Gazebo/Grey</material>

File: src/rove_description/urdf/rove.urdf.xacro (robot description, xacro)
@@ -118,5 +118,5 @@
         <parent link="base_link" />
         <child link="friction_plate_base" />
-        <origin xyz="0.22 0 0.2" rpy="0 0 0" />
+        <origin xyz="0.24 0 0.2" rpy="0 0 0" />
     </joint>
     <!-- <xacro:rove_ros2_control/> -->
