Commit message: Revert "Merge branch 'insta360_x4' into live"
This reverts commit f9a93bf79524257e9d00627eee195e704f7b0d9d, reversing
changes made to 6652aeb3a13d9ec5d9911ca3182db0e179a35409.

File: src/rove_description/urdf/gazebo.urdf.xacro (robot description, xacro)
@@ -34,11 +34,4 @@
         </plugin>
         <plugin filename="gz-sim-navsat-system" name="gz::sim::systems::NavSat"/>
-        <gazebo reference="friction_plate_base">
-            <material>Gazebo/Grey</material>
-            <mu1>100.0</mu1>
-            <mu2>100.0</mu2>
-            <kp>1000000.0</kp>
-            <kd>1.0</kd>
-        </gazebo>
     </gazebo>
 </robot>

File: src/rove_description/urdf/rove.urdf.xacro (robot description, xacro)
@@ -2,11 +2,11 @@
 <robot name="rove" xmlns:xacro="http://www.ros.org/wiki/xacro">
     <material name="rubber_color">
-        <color rgba="0.1 0.1 0.1 1.0" />
+        <color rgba="0.1 0.1 0.1 1.0"/>
     </material>
     <material name="frame_color">
-        <color rgba="0.5 0.5 0.5 1.0" />
+        <color rgba="0.5 0.5 0.5 1.0"/>
     </material>
     <material name="lidar_color">
-        <color rgba="1 0 0 1.0" />
+        <color rgba="1 0 0 1.0"/>
     </material>
     <xacro:include filename="$(find rove_description)/urdf/gazebo.urdf.xacro" />
@@ -18,116 +18,38 @@
     <link name="base_link">
         <visual>
-            <origin xyz="0 0 0" rpy="0 0 0" />
+            <origin xyz="0 0 0" rpy="0 0 0"/>
             <geometry>
-                <mesh
-                    filename="https://raw.githubusercontent.com/clubcapra/rove/main/src/rove_description/meshes/base.stl" />
+                <mesh filename="https://raw.githubusercontent.com/clubcapra/rove/main/src/rove_description/meshes/base.stl"/>
             </geometry>
-            <material name="frame_color" />
+            <material name="frame_color"/>
         </visual>
         <visual>
-            <origin xyz="0 0 0" rpy="0 0 0" />
+            <origin xyz="0 0 0" rpy="0 0 0"/>
             <geometry>
-                <mesh filename="file://$(find rove_description)/meshes/base.stl" />
+                <mesh filename="file://$(find rove_description)/meshes/base.stl"/>
             </geometry>
-            <material name="frame_color" />
+            <material name="frame_color"/>
         </visual>
         <collision>
-            <origin xyz="0 0 0" rpy="0 0 0" />
+            <origin xyz="0 0 0" rpy="0 0 0"/>
             <geometry>
-                <mesh filename="file://$(find rove_description)/meshes/base.stl" />
+                <mesh filename="file://$(find rove_description)/meshes/base.stl"/>
             </geometry>
         </collision>
         <inertial>
-            <origin xyz="0 0 0.5" rpy="0 0 0" />
-            <mass value="80" />
-            <inertia ixx="1" ixy="0" ixz="0" iyy="1" iyz="0" izz="1" />
+            <origin xyz="0 0 0.5" rpy="0 0 0"/>
+            <mass value="80"/>
+            <inertia ixx="1"  ixy="0"  ixz="0" iyy="1" iyz="0" izz="1" />
         </inertial>
     </link>
-    <link name="friction_plate_base">
-        <visual>
-            <origin xyz="0 0 0" rpy="0 0 0" />
-            <geometry>
-                <box size="0.3 0.3 0.01" />
-            </geometry>
-            <material name="frame_color" />
-        </visual>
-        <visual>
-            <origin xyz="0.14 0 0.02" rpy="0 0 0" />
-            <geometry>
-                <box size="0.02 0.3 0.04" />
-            </geometry>
-            <material name="frame_color" />
-        </visual>
-        <visual>
-            <origin xyz="-0.14 0 0.02" rpy="0 0 0" />
-            <geometry>
-                <box size="0.02 0.3 0.04" />
-            </geometry>
-            <material name="frame_color" />
-        </visual>
-        <visual>
-            <origin xyz="0 0.14 0.02" rpy="0 0 0" />
-            <geometry>
-                <box size="0.26 0.02 0.04" />
-            </geometry>
-            <material name="frame_color" />
-        </visual>
-        <visual>
-            <origin xyz="0 -0.14 0.02" rpy="0 0 0" />
-            <geometry>
-                <box size="0.26 0.02 0.04" />
-            </geometry>
-            <material name="frame_color" />
-        </visual>
-        <collision>
-            <origin xyz="0 0 0" rpy="0 0 0" />
-            <geometry>
-                <box size="0.3 0.3 0.01" />
-            </geometry>
-        </collision>
-        <collision>
-            <origin xyz="0.14 0 0.02" rpy="0 0 0" />
-            <geometry>
-                <box size="0.02 0.3 0.04" />
-            </geometry>
-        </collision>
-        <collision>
-            <origin xyz="-0.14 0 0.02" rpy="0 0 0" />
-            <geometry>
-                <box size="0.02 0.3 0.04" />
-            </geometry>
-        </collision>
-        <collision>
-            <origin xyz="0 0.14 0.02" rpy="0 0 0" />
-            <geometry>
-                <box size="0.26 0.02 0.04" />
-            </geometry>
-        </collision>
-        <collision>
-            <origin xyz="0 -0.14 0.02" rpy="0 0 0" />
-            <geometry>
-                <box size="0.26 0.02 0.04" />
-            </geometry>
-        </collision>
-        <inertial>
-            <mass value="1.5" />
-            <inertia ixx="0.02" ixy="0" ixz="0" iyy="0.02" iyz="0" izz="0.02" />
-        </inertial>
-    </link>
-    <joint name="friction_plate_base_joint" type="fixed">
-        <parent link="base_link" />
-        <child link="friction_plate_base" />
-        <origin xyz="0.22 0 0.2" rpy="0 0 0" />
-    </joint>
     <!-- <xacro:rove_ros2_control/> -->
-    <!-- Put these at -1 to mock the motors if working without the motors -->
+     <!-- Put these at -1 to mock the motors if working without the motors -->
     <!-- <xacro:odrive_control fl_id="21" rl_id="22" fr_id="23" rr_id="24"/> -->
     <!-- TODO Fix rr Odrive, it keeps crashing the rest of the drives. IT has been disabled for now. -->
-    <xacro:odrive_control fl_id="21" rl_id="22" fr_id="23" rr_id="24" />
+    <xacro:odrive_control fl_id="21" rl_id="22" fr_id="23" rr_id="-1"/>
     <!-- Insert ovis on top of rove -->
     <!-- <xacro:property name="robot_root" value="base_link" />
     <xacro:property name="ovis_robot_namespace" value="rove" />
     <xacro:property name="ovis_base_origin" value="-0.2 0 0.2" />
-    <xacro:ovis base_parent="${robot_root}" prefix="${ovis_robot_namespace}"
-    joint_base_origin_xyz="${ovis_base_origin}" /> -->
+    <xacro:ovis base_parent="${robot_root}" prefix="${ovis_robot_namespace}" joint_base_origin_xyz="${ovis_base_origin}" /> -->
 </robot>

File: src/rove_description/urdf/sensor.urdf.xacro (robot description, xacro)
@@ -25,5 +25,5 @@
         <visual>
             <geometry>
-                <cylinder length="0.05" radius="0.05" />
+                <cylinder length="0.1" radius="0.1" />
             </geometry>
         </visual>
@@ -31,5 +31,5 @@
             <origin xyz="0 0 0" rpy="0 0 0" />
             <geometry>
-                <cylinder length="0.05" radius="0.05" />
+                <cylinder length="0.1" radius="0.1" />
             </geometry>
         </collision>
@@ -42,5 +42,5 @@
         <visual>
             <geometry>
-                <cylinder length="0.05" radius="0.05" />
+                <cylinder length="0.1" radius="0.1" />
             </geometry>
         </visual>
@@ -48,5 +48,5 @@
             <origin xyz="0 0 0" rpy="0 0 0" />
             <geometry>
-                <cylinder length="0.05" radius="0.05" />
+                <cylinder length="0.1" radius="0.1" />
             </geometry>
         </collision>
@@ -61,5 +61,5 @@
             <origin xyz="0 0 0" rpy="0 0 0" />
             <geometry>
-                <cylinder length="0.05" radius="0.05" />
+                <cylinder length="0.1" radius="0.1" />
             </geometry>
         </visual>
@@ -67,5 +67,5 @@
             <origin xyz="0 0 0" rpy="0 0 0" />
             <geometry>
-                <cylinder length="0.05" radius="0.05" />
+                <cylinder length="0.1" radius="0.1" />
             </geometry>
         </collision>
