Commit message: update: temporary rove urdf - update the lidar - update sensors - del gazebo - del old mesh

File: src/rove_description/urdf/livox.urdf.xacro (robot description, xacro)
@@ -1,5 +1,5 @@
 <?xml version="1.0"?>
 <robot xmlns:xacro="http://www.ros.org/wiki/xacro">
-  <xacro:macro name="velodyne_lidar" params="name parent_link *origin
+  <xacro:macro name="livox_lidar" params="name parent_link *origin
                                              ang_res_h:=0.4 min_ang_h:=-3.141592 max_ang_h:=3.141592
                                              ang_res_v:=2.0 min_ang_v:=-0.261799 max_ang_v:=0.261799
@@ -18,16 +18,10 @@
       <visual>
         <geometry>
-          <mesh filename="file://$(find rove_description)/meshes/vlp16/VLP16_base_1.dae"/>
-        </geometry>
-      </visual>
-      <visual>
-        <geometry>
-          <mesh filename="file://$(find rove_description)/meshes/vlp16/VLP16_base_2.dae"/>
+          <box size="0.06 0.06 0.06"/>
         </geometry>
       </visual>
       <collision>
-        <origin rpy="0 0 0" xyz="0 0 0.03585"/>
         <geometry>
-          <cylinder radius="0.0516" length="0.0717"/>
+          <box size="0.06 0.06 0.06"/>
         </geometry>
       </collision>
@@ -56,36 +50,6 @@
       <child link="${name}_laser"/>
     </joint>
-    <xacro:property name="samples_h" value="${round((max_ang_h - min_ang_h) * 180 / (ang_res_h * pi))}"/>
-    <xacro:property name="samples_v" value="${round((max_ang_v - min_ang_v) * 180 / (ang_res_v * pi))}"/>
-    <gazebo reference="${name}_laser">
-      <sensor name="${name}" type="gpu_lidar">
-        <visualize>true</visualize>
-        <always_on>true</always_on>
-        <update_rate>50</update_rate>
-        <topic>scan</topic>
-        <gz_frame_id>${name}_laser</gz_frame_id>
-        <lidar>
-          <scan>
-            <horizontal>
-              <samples>${samples_h}</samples>
-              <resolution>1</resolution>
-              <min_angle>${min_ang_h}</min_angle>
-              <max_angle>${max_ang_h}</max_angle>
-            </horizontal>
-            <vertical>
-              <samples>${samples_v}</samples>
-              <resolution>1</resolution>
-              <min_angle>${min_ang_v}</min_angle>
-              <max_angle>${max_ang_v}</max_angle>
-            </vertical>
-          </scan>
-          <range>
-            <min>${min_range}</min>
-            <max>${max_range}</max>
-            <resolution>0.01</resolution>
-          </range>
-        </lidar>
-      </sensor>
-    </gazebo>
+    <xacro:property name="samples_h" value="${floor((max_ang_h - min_ang_h) * 180 / (ang_res_h * pi) + 0.5)}"/>
+    <xacro:property name="samples_v" value="${floor((max_ang_v - min_ang_v) * 180 / (ang_res_v * pi) + 0.5)}"/>
   </xacro:macro>
 </robot>

File: src/rove_description/urdf/sensor.urdf.xacro (robot description, xacro)
@@ -2,19 +2,16 @@
 <robot xmlns:xacro="http://www.ros.org/wiki/xacro">
     <xacro:property name="M_PI" value="3.1415926535897931" />
-    <xacro:include filename="$(find rove_description)/urdf/velodyne.urdf.xacro" />
-    <joint name="sensor_joint" type="fixed">
+    <xacro:include filename="$(find rove_description)/urdf/livox.urdf.xacro" />
+    <joint name="top_joint" type="fixed">
         <parent link="base_link" />
-        <child link="sensor_link" />
-        <origin xyz="-0.3 0 0.4" rpy="0 0 0" />
+        <child link="top_link"/>
+        <origin xyz="0 0 0.15" rpy="0 0 0"/>
     </joint>
-    <joint name="zed_camera_joint" type="fixed">
-        <parent link="sensor_link" />
-        <child link="zed_camera_link" />
-        <origin xyz="0.1 0 0" rpy="0 0 0" />
-    </joint>
+    <link name="top_link">
+    </link>
     <joint name="camera_joint" type="fixed">
-        <parent link="sensor_link" />
+        <parent link="top_link" />
         <child link="camera_link" />
-        <origin xyz="0.1 0 0" rpy="-1.57 0 -1.57" />
+        <origin xyz="-0.4 0 0" rpy="0 0 ${pi}" />
     </joint>
     <link name="camera_link">
@@ -25,103 +22,15 @@
         <visual>
             <geometry>
-                <cylinder length="0.05" radius="0.05" />
+                <box size="0.05 0.05 0.05"/>
             </geometry>
         </visual>
         <collision>
-            <origin xyz="0 0 0" rpy="0 0 0" />
             <geometry>
-                <cylinder length="0.05" radius="0.05" />
+                <box size="0.05 0.05 0.05"/>
             </geometry>
         </collision>
     </link>
-    <link name="zed_camera_link">
-        <inertial>
-            <mass value="0.1" />
-            <inertia ixx="0.0001" ixy="0.0" ixz="0.0" iyy="0.0001" iyz="0.0" izz="0.0001" />
-        </inertial>
-        <visual>
-            <geometry>
-                <cylinder length="0.05" radius="0.05" />
-            </geometry>
-        </visual>
-        <collision>
-            <origin xyz="0 0 0" rpy="0 0 0" />
-            <geometry>
-                <cylinder length="0.05" radius="0.05" />
-            </geometry>
-        </collision>
-    </link>
-    <link name="sensor_link">
-        <inertial>
-            <origin xyz="0 0 0" rpy="0 0 0" />
-            <mass value="0.1" />
-            <inertia ixx="0.0001" ixy="0.0" ixz="0.0" iyy="0.0001" iyz="0.0" izz="0.0001" />
-        </inertial>
-        <visual>
-            <origin xyz="0 0 0" rpy="0 0 0" />
-            <geometry>
-                <cylinder length="0.05" radius="0.05" />
-            </geometry>
-        </visual>
-        <collision>
-            <origin xyz="0 0 0" rpy="0 0 0" />
-            <geometry>
-                <cylinder length="0.05" radius="0.05" />
-            </geometry>
-        </collision>
-    </link>
-    <xacro:velodyne_lidar name="velodyne" parent_link="base_link">
-        <origin xyz="-0.2 0.0 0.5" rpy="0 0 ${-pi/2}" />
-    </xacro:velodyne_lidar>
-    <gazebo reference="sensor_link">
-        <material>Gazebo/Black</material>
-        <sensor name="imu_sensor" type="imu">
-            <gz_frame_id>sensor_link</gz_frame_id>
-            <always_on>true</always_on>
-            <update_rate>50</update_rate>
-            <topic>imu</topic>
-        </sensor>
-        <sensor name="gps_sensor" type="navsat">
-            <gz_frame_id>sensor_link</gz_frame_id>
-            <always_on>true</always_on>
-            <update_rate>1</update_rate>
-            <topic>navsat</topic>
-        </sensor>
-        <sensor name="depth_camera1" type="depth_camera">
-            <gz_frame_id>camera_link</gz_frame_id>
-            <update_rate>10</update_rate>
-            <topic>depth_camera</topic>
-            <camera>
-                <horizontal_fov>1.88</horizontal_fov>
-                <image>
-                    <width>1344</width>
-                    <height>376</height>
-                    <format>R_FLOAT32</format>
-                </image>
-                <clip>
-                    <near>0.5</near>
-                    <far>20.0</far>
-                </clip>
-                <!-- Rotate the camera to point forward -->
-                <origin xyz="0.1 0 0.4" rpy="${-pi/2} 0 ${-pi/2}" />
-            </camera>
-        </sensor>
-        <sensor name="camera1" type="camera">
-            <gz_frame_id>camera_link</gz_frame_id>
-            <update_rate>10</update_rate>
-            <topic>camera</topic>
-            <camera>
-                <horizontal_fov>1.88</horizontal_fov>
-                <image>
-                    <width>1344</width>
-                    <height>376</height>
-                    <format>R_FLOAT32</format>
-                </image>
-                <clip>
-                    <near>0.5</near>
-                    <far>20.0</far>
-                </clip>
-            </camera>
-        </sensor>
-    </gazebo>
+    <xacro:livox_lidar name="livox" parent_link="top_link">
+        <origin xyz="-0.3 0.0 0.13" rpy="0.5235987755983  0 ${-pi/2}" />
+    </xacro:livox_lidar>
 </robot>
