Commit message: add zed simulation

File: src/rove_description/urdf/sensor.urdf.xacro (robot description, xacro)
@@ -4,24 +4,24 @@
     <xacro:include filename="$(find rove_description)/urdf/velodyne.urdf.xacro" />
     <joint name="sensor_joint" type="fixed">
-        <parent link="base_link"/>
-        <child link="sensor_link"/>
-        <origin xyz="0.1 0 0.212" rpy="0 0 0"/>
+        <parent link="base_link" />
+        <child link="sensor_link" />
+        <origin xyz="0.1 0 0.4" rpy="0 0 0" />
     </joint>
     <link name="sensor_link">
         <inertial>
-            <origin xyz="0 0 0" rpy="0 0 0"/>
-            <mass value="0.1"/>
-            <inertia ixx="0.0001" ixy="0.0" ixz="0.0" iyy="0.0001" iyz="0.0" izz="0.0001"/>
+            <origin xyz="0 0 0" rpy="0 0 0" />
+            <mass value="0.1" />
+            <inertia ixx="0.0001" ixy="0.0" ixz="0.0" iyy="0.0001" iyz="0.0" izz="0.0001" />
         </inertial>
         <visual>
-            <origin xyz="0 0 0" rpy="0 0 0"/>
+            <origin xyz="0 0 0" rpy="0 0 0" />
             <geometry>
-                <cylinder length="0.1" radius="0.1"/>
+                <cylinder length="0.1" radius="0.1" />
             </geometry>
         </visual>
         <collision>
-            <origin xyz="0 0 0" rpy="0 0 0"/>
+            <origin xyz="0 0 0" rpy="0 0 0" />
             <geometry>
-                <cylinder length="0.1" radius="0.1"/>
+                <cylinder length="0.1" radius="0.1" />
             </geometry>
         </collision>
@@ -44,4 +44,38 @@
             <topic>navsat</topic>
         </sensor>
+        <sensor name="depth_camera1" type="depth_camera">
+            <gz_frame_id>sensor_link</gz_frame_id>
+            <update_rate>10</update_rate>
+            <topic>depth_camera</topic>
+            <camera>
+                <horizontal_fov>1.88</horizontal_fov>
+                <image>
+                    <width>256</width>
+                    <height>256</height>
+                    <format>R_FLOAT32</format>
+                </image>
+                <clip>
+                    <near>0.5</near>
+                    <far>20.0</far>
+                </clip>
+            </camera>
+        </sensor>
+        <sensor name="camera1" type="camera">
+            <gz_frame_id>sensor_link</gz_frame_id>
+            <update_rate>10</update_rate>
+            <topic>camera</topic>
+            <camera>
+                <horizontal_fov>1.88</horizontal_fov>
+                <image>
+                    <width>256</width>
+                    <height>256</height>
+                    <format>R_FLOAT32</format>
+                </image>
+                <clip>
+                    <near>0.5</near>
+                    <far>20.0</far>
+                </clip>
+            </camera>
+        </sensor>
     </gazebo>
 </robot>

Commit message: add 3d color camera + parcours

File: src/rove_description/urdf/sensor.urdf.xacro (robot description, xacro)
@@ -8,4 +8,28 @@
         <origin xyz="0.1 0 0.4" rpy="0 0 0" />
     </joint>
+    <joint name="camera_joint" type="fixed">
+        <parent link="sensor_link" />
+        <child link="camera_link" />
+        <origin xyz="0.1 0 0.4" rpy="-1.57 0 -1.57" />
+    </joint>
+    <link name="camera_link">
+        <inertial>
+            <origin xyz="0 0 0" rpy="0 0 0" />
+            <mass value="0.1" />
+            <inertia ixx="0.0001" ixy="0.0" ixz="0.0" iyy="0.0001" iyz="0.0" izz="0.0001" />
+        </inertial>
+        <visual>
+            <origin xyz="0 0 0" rpy="0 0 0" />
+            <geometry>
+                <cylinder length="0.1" radius="0.1" />
+            </geometry>
+        </visual>
+        <collision>
+            <origin xyz="0 0 0" rpy="0 0 0" />
+            <geometry>
+                <cylinder length="0.1" radius="0.1" />
+            </geometry>
+        </collision>
+    </link>
     <link name="sensor_link">
         <inertial>
@@ -45,5 +69,5 @@
         </sensor>
         <sensor name="depth_camera1" type="depth_camera">
-            <gz_frame_id>sensor_link</gz_frame_id>
+            <gz_frame_id>camera_link</gz_frame_id>
             <update_rate>10</update_rate>
             <topic>depth_camera</topic>
@@ -59,8 +83,10 @@
                     <far>20.0</far>
                 </clip>
+                <!-- Rotate the camera to point forward -->
+                <origin xyz="0.1 0 0.4" rpy="-1.57 0 -1.57" />
             </camera>
         </sensor>
         <sensor name="camera1" type="camera">
-            <gz_frame_id>sensor_link</gz_frame_id>
+            <gz_frame_id>camera_link</gz_frame_id>
             <update_rate>10</update_rate>
             <topic>camera</topic>

Commit message: modification for real hardware

File: src/rove_description/urdf/sensor.urdf.xacro (robot description, xacro)
@@ -8,4 +8,9 @@
         <origin xyz="0.1 0 0.4" rpy="0 0 0" />
     </joint>
+    <joint name="zed_camera_joint" type="fixed">
+        <parent link="sensor_link" />
+        <child link="zed_camera_link" />
+        <origin xyz="0.1 0 0" rpy="0 0 0" />
+    </joint>
     <joint name="camera_joint" type="fixed">
         <parent link="sensor_link" />
@@ -14,4 +19,21 @@
     </joint>
     <link name="camera_link">
+        <inertial>
+            <mass value="0.1" />
+            <inertia ixx="0.0001" ixy="0.0" ixz="0.0" iyy="0.0001" iyz="0.0" izz="0.0001" />
+        </inertial>
+        <visual>
+            <geometry>
+                <cylinder length="0.1" radius="0.1" />
+            </geometry>
+        </visual>
+        <collision>
+            <origin xyz="0 0 0" rpy="0 0 0" />
+            <geometry>
+                <cylinder length="0.1" radius="0.1" />
+            </geometry>
+        </collision>
+    </link>
+    <link name="zed_camera_link">
         <inertial>
             <mass value="0.1" />

Commit message: ROBOT MOVEDDDDD Changed the position of the sensors in the URDF (they wer showed as if they were in the front instead of the back) Modified the inputs for slam

File: src/rove_description/urdf/sensor.urdf.xacro (robot description, xacro)
@@ -6,15 +6,15 @@
         <parent link="base_link" />
         <child link="sensor_link" />
-        <origin xyz="0.1 0 0.4" rpy="0 0 0" />
+        <origin xyz="-0.1 0 0.4" rpy="0 0 0" />
     </joint>
     <joint name="zed_camera_joint" type="fixed">
         <parent link="sensor_link" />
         <child link="zed_camera_link" />
-        <origin xyz="0.1 0 0" rpy="0 0 0" />
+        <origin xyz="-0.1 0 0" rpy="0 0 0" />
     </joint>
     <joint name="camera_joint" type="fixed">
         <parent link="sensor_link" />
         <child link="camera_link" />
-        <origin xyz="0.1 0 0" rpy="-1.57 0 -1.57" />
+        <origin xyz="-0.1 0 0" rpy="-1.57 0 -1.57" />
     </joint>
     <link name="camera_link">
@@ -72,5 +72,5 @@
     </link>
     <xacro:velodyne_lidar name="velodyne" parent_link="base_link">
-        <origin xyz="0.0 0.0 0.4" rpy="0 3.141592 0" />
+        <origin xyz="0.0 0.0 0.4" rpy="0 0 3.1416" />
     </xacro:velodyne_lidar>
     <gazebo reference="sensor_link">

Commit message: add ovis integration

File: src/rove_description/urdf/sensor.urdf.xacro (robot description, xacro)
@@ -6,5 +6,5 @@
         <parent link="base_link" />
         <child link="sensor_link" />
-        <origin xyz="0.1 0 0.4" rpy="0 0 0" />
+        <origin xyz="-0.3 0 0.4" rpy="0 0 0" />
     </joint>
     <joint name="zed_camera_joint" type="fixed">
@@ -25,5 +25,5 @@
         <visual>
             <geometry>
-                <cylinder length="0.1" radius="0.1" />
+                <cylinder length="0.05" radius="0.05" />
             </geometry>
         </visual>
@@ -31,5 +31,5 @@
             <origin xyz="0 0 0" rpy="0 0 0" />
             <geometry>
-                <cylinder length="0.1" radius="0.1" />
+                <cylinder length="0.05" radius="0.05" />
             </geometry>
         </collision>
@@ -42,5 +42,5 @@
         <visual>
             <geometry>
-                <cylinder length="0.1" radius="0.1" />
+                <cylinder length="0.05" radius="0.05" />
             </geometry>
         </visual>
@@ -48,5 +48,5 @@
             <origin xyz="0 0 0" rpy="0 0 0" />
             <geometry>
-                <cylinder length="0.1" radius="0.1" />
+                <cylinder length="0.05" radius="0.05" />
             </geometry>
         </collision>
@@ -61,5 +61,5 @@
             <origin xyz="0 0 0" rpy="0 0 0" />
             <geometry>
-                <cylinder length="0.1" radius="0.1" />
+                <cylinder length="0.05" radius="0.05" />
             </geometry>
         </visual>
@@ -67,10 +67,10 @@
             <origin xyz="0 0 0" rpy="0 0 0" />
             <geometry>
-                <cylinder length="0.1" radius="0.1" />
+                <cylinder length="0.05" radius="0.05" />
             </geometry>
         </collision>
     </link>
     <xacro:velodyne_lidar name="velodyne" parent_link="base_link">
-        <origin xyz="0.0 0.0 0.4" rpy="0 0 0" />
+        <origin xyz="-0.2 0.0 0.5" rpy="0 0 0" />
     </xacro:velodyne_lidar>
     <gazebo reference="sensor_link">

Commit message: Live (#80)
* Trying to fix udevrules for vectornav
Changed velodyne orientation to offset it 180deg.
This will probably have an impact in the simulation in gazebo.

Adjusted the launch script to stop can bus on exit.

Disabled odrive id 24 rr_track (rear right track).

Disabled slam_3d to simplify testing.

* ROBOT MOVEDDDDD
Changed the position of the sensors in the URDF (they wer showed as if they were in the front instead of the back)
Modified the inputs for slam

---------

Co-authored-by: nathan-gt <nathan.gt.protic@gmail.com>

File: src/rove_description/urdf/sensor.urdf.xacro (robot description, xacro)
@@ -6,15 +6,15 @@
         <parent link="base_link" />
         <child link="sensor_link" />
-        <origin xyz="-0.3 0 0.4" rpy="0 0 0" />
+        <origin xyz="-0.1 0 0.4" rpy="0 0 0" />
     </joint>
     <joint name="zed_camera_joint" type="fixed">
         <parent link="sensor_link" />
         <child link="zed_camera_link" />
-        <origin xyz="0.1 0 0" rpy="0 0 0" />
+        <origin xyz="-0.1 0 0" rpy="0 0 0" />
     </joint>
     <joint name="camera_joint" type="fixed">
         <parent link="sensor_link" />
         <child link="camera_link" />
-        <origin xyz="0.1 0 0" rpy="-1.57 0 -1.57" />
+        <origin xyz="-0.1 0 0" rpy="-1.57 0 -1.57" />
     </joint>
     <link name="camera_link">
@@ -72,5 +72,5 @@
     </link>
     <xacro:velodyne_lidar name="velodyne" parent_link="base_link">
-        <origin xyz="-0.2 0.0 0.5" rpy="0 0 0" />
+        <origin xyz="0.0 0.0 0.4" rpy="0 0 3.1416" />
     </xacro:velodyne_lidar>
     <gazebo reference="sensor_link">

Commit message: Revert "ROBOT MOVEDDDDD"
This reverts commit 6652aeb3a13d9ec5d9911ca3182db0e179a35409.

File: src/rove_description/urdf/sensor.urdf.xacro (robot description, xacro)
@@ -6,15 +6,15 @@
         <parent link="base_link" />
         <child link="sensor_link" />
-        <origin xyz="-0.1 0 0.4" rpy="0 0 0" />
+        <origin xyz="0.1 0 0.4" rpy="0 0 0" />
     </joint>
     <joint name="zed_camera_joint" type="fixed">
         <parent link="sensor_link" />
         <child link="zed_camera_link" />
-        <origin xyz="-0.1 0 0" rpy="0 0 0" />
+        <origin xyz="0.1 0 0" rpy="0 0 0" />
     </joint>
     <joint name="camera_joint" type="fixed">
         <parent link="sensor_link" />
         <child link="camera_link" />
-        <origin xyz="-0.1 0 0" rpy="-1.57 0 -1.57" />
+        <origin xyz="0.1 0 0" rpy="-1.57 0 -1.57" />
     </joint>
     <link name="camera_link">
@@ -72,5 +72,5 @@
     </link>
     <xacro:velodyne_lidar name="velodyne" parent_link="base_link">
-        <origin xyz="0.0 0.0 0.4" rpy="0 0 3.1416" />
+        <origin xyz="0.0 0.0 0.4" rpy="0 3.141592 0" />
     </xacro:velodyne_lidar>
     <gazebo reference="sensor_link">

Commit message: Revert "Insta360 x4 featuring pan zoom (#81)"
This reverts commit 61630af2df00eae05ed70acb7f14a6c00dfddfb0.

File: src/rove_description/urdf/sensor.urdf.xacro (robot description, xacro)
@@ -6,15 +6,15 @@
         <parent link="base_link" />
         <child link="sensor_link" />
-        <origin xyz="-0.1 0 0.4" rpy="0 0 0" />
+        <origin xyz="-0.3 0 0.4" rpy="0 0 0" />
     </joint>
     <joint name="zed_camera_joint" type="fixed">
         <parent link="sensor_link" />
         <child link="zed_camera_link" />
-        <origin xyz="-0.1 0 0" rpy="0 0 0" />
+        <origin xyz="0.1 0 0" rpy="0 0 0" />
     </joint>
     <joint name="camera_joint" type="fixed">
         <parent link="sensor_link" />
         <child link="camera_link" />
-        <origin xyz="-0.1 0 0" rpy="-1.57 0 -1.57" />
+        <origin xyz="0.1 0 0" rpy="-1.57 0 -1.57" />
     </joint>
     <link name="camera_link">
@@ -72,5 +72,5 @@
     </link>
     <xacro:velodyne_lidar name="velodyne" parent_link="base_link">
-        <origin xyz="0.0 0.0 0.4" rpy="0 0 3.1416" />
+        <origin xyz="-0.2 0.0 0.5" rpy="0 0 0" />
     </xacro:velodyne_lidar>
     <gazebo reference="sensor_link">

Commit message: changing var for real world

File: src/rove_description/urdf/sensor.urdf.xacro (robot description, xacro)
@@ -16,5 +16,5 @@
         <parent link="sensor_link" />
         <child link="camera_link" />
-        <origin xyz="-0.1 0 0" rpy="-1.57 0 -1.57" />
+        <origin xyz="-0.1 0 0" rpy="-1.57 0 ${-pi/2}" />
     </joint>
     <link name="camera_link">
@@ -72,5 +72,5 @@
     </link>
     <xacro:velodyne_lidar name="velodyne" parent_link="base_link">
-        <origin xyz="0.0 0.0 0.4" rpy="0 0 3.1416" />
+        <origin xyz="0.0 0.0 0.4" rpy="0 0 ${-pi/2}" />
     </xacro:velodyne_lidar>
     <gazebo reference="sensor_link">
@@ -104,5 +104,5 @@
                 </clip>
                 <!-- Rotate the camera to point forward -->
-                <origin xyz="0.1 0 0.4" rpy="-1.57 0 -1.57" />
+                <origin xyz="0.1 0 0.4" rpy="${-pi/2} 0 ${-pi/2}" />
             </camera>
         </sensor>

Commit message: forgotten value

File: src/rove_description/urdf/sensor.urdf.xacro (robot description, xacro)
@@ -16,5 +16,5 @@
         <parent link="sensor_link" />
         <child link="camera_link" />
-        <origin xyz="-0.1 0 0" rpy="-1.57 0 ${-pi/2}" />
+        <origin xyz="-0.1 0 0" rpy="${-pi/2} 0 ${-pi/2}" />
     </joint>
     <link name="camera_link">

Commit message: Fixed some issues

File: src/rove_description/urdf/sensor.urdf.xacro (robot description, xacro)
@@ -72,5 +72,5 @@
     </link>
     <xacro:velodyne_lidar name="velodyne" parent_link="base_link">
-        <origin xyz="0.0 0.0 0.4" rpy="0 0 3.1416" />
+        <origin xyz="0.0 0.0 0.4" rpy="0 0 -1.5707963" />
     </xacro:velodyne_lidar>
     <gazebo reference="sensor_link">

Commit message: update: add imu in urdf

File: src/rove_description/urdf/sensor.urdf.xacro (robot description, xacro)
@@ -9,4 +9,25 @@
     </joint>
     <link name="top_link">
+    </link>
+    <joint name="imu_joint" type="fixed">
+        <parent link="top_link" />
+        <child link="camera_link" />
+        <origin xyz="-0.05 0.15 -0.06" rpy="0 0 0" />
+    </joint>
+    <link name="imu_link">
+        <inertial>
+            <mass value="0.1" />
+            <inertia ixx="0.0001" ixy="0.0" ixz="0.0" iyy="0.0001" iyz="0.0" izz="0.0001" />
+        </inertial>
+        <visual>
+            <geometry>
+                <box size="0.05 0.05 0.01"/>
+            </geometry>
+        </visual>
+        <collision>
+            <geometry>
+                <box size="0.05 0.05 0.01"/>
+            </geometry>
+        </collision>
     </link>
     <joint name="camera_joint" type="fixed">
