Commit message: Joy or cmd_vel are lagging

File: src/rove_description/urdf/rove.urdf.xacro (robot description, xacro)
@@ -15,5 +15,6 @@
     <xacro:include filename="$(find rove_description)/urdf/flipper.urdf.xacro" />
     <xacro:include filename="$(find rove_description)/urdf/track.urdf.xacro" />
-    <xacro:include filename="$(find ovis_description)/urdf/ovis.urdf.xacro" />
+    <xacro:include filename="$(find rove_description)/urdf/rove.ros2_control.urdf.xacro" />
+    <!-- <xacro:include filename="$(find ovis_description)/urdf/ovis.urdf.xacro" /> -->
     <link name="base_footprint"/>
     <link name="base_link">
@@ -42,8 +43,10 @@
         <child link="base_link"/>
     </joint>
+    <!-- <xacro:rove_ros2_control/> -->
+    <xacro:odrive_control fl_id="0" rl_id="-1" fr_id="-1" rr_id="-1"/>
     <!-- Insert ovis on top of rove -->
-    <xacro:property name="robot_root" value="base_link" />
+    <!-- <xacro:property name="robot_root" value="base_link" />
     <xacro:property name="ovis_robot_namespace" value="rove" />
     <xacro:property name="ovis_base_origin" value="-0.2 0 0.2" />
-    <xacro:ovis base_parent="${robot_root}" prefix="${ovis_robot_namespace}" joint_base_origin_xyz="${ovis_base_origin}" />
+    <xacro:ovis base_parent="${robot_root}" prefix="${ovis_robot_namespace}" joint_base_origin_xyz="${ovis_base_origin}" /> -->
 </robot>

File: src/rove_description/urdf/track.urdf.xacro (robot description, xacro)
@@ -16,4 +16,20 @@
             <parent link="base_link"/>
             <child link="track_${suffix}"/>
+        </joint>
+        <joint name="track_f${suffix}_j" type="fixed">
+            <origin xyz="${joint_origin}" rpy="0 0 0 "/>
+            <parent link="track_${suffix}"/>
+            <child link="track_f${suffix}"/>
+            <!-- <axis xyz="0 1 0"/>
+            <dynamics damping="0.2"/>
+            <limit effort="100" velocity="1.0"/> -->
+        </joint>
+        <joint name="track_r${suffix}_j" type="fixed">
+            <origin xyz="${joint_origin}" rpy="0 0 0 "/>
+            <parent link="track_${suffix}"/>
+            <child link="track_r${suffix}"/>
+            <!-- <axis xyz="0 -1 0"/>
+            <dynamics damping="0.2"/>
+            <limit effort="100" velocity="1.0"/> -->
         </joint>
         <link name="track_${suffix}">
@@ -50,4 +66,18 @@
             </inertial>
         </link>
+        <link name="track_f${suffix}">
+            <inertial>
+                <origin xyz="0 0 0" rpy="0 0 0"/>
+                <mass value="1"/>
+                <inertia ixx="100"  ixy="0"  ixz="0" iyy="100" iyz="0" izz="100" />
+            </inertial>
+        </link>
+        <link name="track_r${suffix}">
+            <inertial>
+                <origin xyz="0 0 0" rpy="0 0 0"/>
+                <mass value="1"/>
+                <inertia ixx="100"  ixy="0"  ixz="0" iyy="100" iyz="0" izz="100" />
+            </inertial>
+        </link>
         <gazebo>
             <plugin name='gz::sim::systems::TrackController' filename='libignition-gazebo-track-controller-system.so'>

Commit message: add real imu + lidar mapping

File: src/rove_description/urdf/rove.urdf.xacro (robot description, xacro)
@@ -11,5 +11,4 @@
     </material>
     <xacro:include filename="$(find rove_description)/urdf/gazebo.urdf.xacro" />
-    <xacro:include filename="$(find rove_description)/urdf/lidar.urdf.xacro" />
     <xacro:include filename="$(find rove_description)/urdf/sensor.urdf.xacro" />
     <xacro:include filename="$(find rove_description)/urdf/flipper.urdf.xacro" />

File: src/rove_description/urdf/sensor.urdf.xacro (robot description, xacro)
@@ -1,4 +1,6 @@
 <?xml version="1.0"?>
 <robot xmlns:xacro="http://www.ros.org/wiki/xacro">
+    <xacro:property name="M_PI" value="3.1415926535897931" />
+    <xacro:include filename="$(find rove_description)/urdf/velodyne.urdf.xacro" />
     <joint name="sensor_joint" type="fixed">
         <parent link="base_link"/>
@@ -25,4 +27,7 @@
         </collision>
     </link>
+    <xacro:velodyne_lidar name="velodyne" parent_link="base_link">
+        <origin xyz="0.0 0.0 0.4" rpy="0 0 0" />
+    </xacro:velodyne_lidar>
     <gazebo reference="sensor_link">
         <material>Gazebo/Black</material>

Commit message: add ovis arm support

File: src/rove_description/urdf/rove.urdf.xacro (robot description, xacro)
@@ -2,11 +2,11 @@
 <robot name="rove" xmlns:xacro="http://www.ros.org/wiki/xacro">
     <material name="rubber_color">
-        <color rgba="0.1 0.1 0.1 1.0"/>
+        <color rgba="0.1 0.1 0.1 1.0" />
     </material>
     <material name="frame_color">
-        <color rgba="0.5 0.5 0.5 1.0"/>
+        <color rgba="0.5 0.5 0.5 1.0" />
     </material>
     <material name="lidar_color">
-        <color rgba="1 0 0 1.0"/>
+        <color rgba="1 0 0 1.0" />
     </material>
     <xacro:include filename="$(find rove_description)/urdf/gazebo.urdf.xacro" />
@@ -15,40 +15,36 @@
     <xacro:include filename="$(find rove_description)/urdf/track.urdf.xacro" />
     <xacro:include filename="$(find rove_description)/urdf/rove.ros2_control.urdf.xacro" />
-    <!-- <xacro:include filename="$(find ovis_description)/urdf/ovis.urdf.xacro" /> -->
     <link name="base_link">
         <visual>
-            <origin xyz="0 0 0" rpy="0 0 0"/>
+            <origin xyz="0 0 0" rpy="0 0 0" />
             <geometry>
-                <mesh filename="https://raw.githubusercontent.com/clubcapra/rove/main/src/rove_description/meshes/base.stl"/>
+                <mesh
+                    filename="https://raw.githubusercontent.com/clubcapra/rove/main/src/rove_description/meshes/base.stl" />
             </geometry>
-            <material name="frame_color"/>
+            <material name="frame_color" />
         </visual>
         <visual>
-            <origin xyz="0 0 0" rpy="0 0 0"/>
+            <origin xyz="0 0 0" rpy="0 0 0" />
             <geometry>
-                <mesh filename="file://$(find rove_description)/meshes/base.stl"/>
+                <mesh filename="file://$(find rove_description)/meshes/base.stl" />
             </geometry>
-            <material name="frame_color"/>
+            <material name="frame_color" />
         </visual>
         <collision>
-            <origin xyz="0 0 0" rpy="0 0 0"/>
+            <origin xyz="0 0 0" rpy="0 0 0" />
             <geometry>
-                <mesh filename="file://$(find rove_description)/meshes/base.stl"/>
+                <mesh filename="file://$(find rove_description)/meshes/base.stl" />
             </geometry>
         </collision>
         <inertial>
-            <origin xyz="0 0 0.5" rpy="0 0 0"/>
-            <mass value="80"/>
-            <inertia ixx="1"  ixy="0"  ixz="0" iyy="1" iyz="0" izz="1" />
+            <origin xyz="0 0 0.5" rpy="0 0 0" />
+            <mass value="80" />
+            <inertia ixx="1" ixy="0" ixz="0" iyy="1" iyz="0" izz="1" />
         </inertial>
     </link>
     <!-- <xacro:rove_ros2_control/> -->
-     <!-- Put these at -1 to mock the motors if working without the motors -->
+    <!-- Put these at -1 to mock the motors if working without the motors -->
     <!-- <xacro:odrive_control fl_id="21" rl_id="22" fr_id="23" rr_id="24"/> -->
-    <xacro:odrive_control fl_id="21" rl_id="22" fr_id="23" rr_id="24"/>
-    <!-- Insert ovis on top of rove -->
-    <!-- <xacro:property name="robot_root" value="base_link" />
-    <xacro:property name="ovis_robot_namespace" value="rove" />
-    <xacro:property name="ovis_base_origin" value="-0.2 0 0.2" />
-    <xacro:ovis base_parent="${robot_root}" prefix="${ovis_robot_namespace}" joint_base_origin_xyz="${ovis_base_origin}" /> -->
+    <xacro:odrive_control fl_id="21" rl_id="22" fr_id="23" rr_id="24" />
+    <xacro:property name="robot_root" value="base_link" />
 </robot>

File: src/rove_description/urdf/sensor.urdf.xacro (robot description, xacro)
@@ -6,5 +6,5 @@
         <parent link="base_link" />
         <child link="sensor_link" />
-        <origin xyz="0.1 0 0.4" rpy="0 0 0" />
+        <origin xyz="0.3 0 0.4" rpy="0 0 0" />
     </joint>
     <joint name="zed_camera_joint" type="fixed">
@@ -72,5 +72,5 @@
     </link>
     <xacro:velodyne_lidar name="velodyne" parent_link="base_link">
-        <origin xyz="0.0 0.0 0.4" rpy="0 0 0" />
+        <origin xyz="0.3 0.0 0.4" rpy="0 0 0" />
     </xacro:velodyne_lidar>
     <gazebo reference="sensor_link">

Commit message: Trying to fix udevrules for vectornav Changed velodyne orientation to offset it 180deg. This will probably have an impact in the simulation in gazebo.
Adjusted the launch script to stop can bus on exit.

Disabled odrive id 24 rr_track (rear right track).

Disabled slam_3d to simplify testing.

File: src/rove_description/urdf/rove.urdf.xacro (robot description, xacro)
@@ -47,5 +47,5 @@
     <!-- <xacro:odrive_control fl_id="21" rl_id="22" fr_id="23" rr_id="24"/> -->
     <!-- TODO Fix rr Odrive, it keeps crashing the rest of the drives. IT has been disabled for now. -->
-    <xacro:odrive_control fl_id="21" rl_id="22" fr_id="23" rr_id="24"/>
+    <xacro:odrive_control fl_id="21" rl_id="22" fr_id="23" rr_id="-1"/>
     <!-- Insert ovis on top of rove -->
     <!-- <xacro:property name="robot_root" value="base_link" />

File: src/rove_description/urdf/sensor.urdf.xacro (robot description, xacro)
@@ -72,5 +72,5 @@
     </link>
     <xacro:velodyne_lidar name="velodyne" parent_link="base_link">
-        <origin xyz="0.0 0.0 0.4" rpy="0 0 0" />
+        <origin xyz="0.0 0.0 0.4" rpy="0 3.141592 0" />
     </xacro:velodyne_lidar>
     <gazebo reference="sensor_link">

Commit message: change ovis origin

File: src/rove_description/urdf/rove.urdf.xacro (robot description, xacro)
@@ -118,5 +118,5 @@
         <parent link="base_link" />
         <child link="friction_plate_base" />
-        <origin xyz="0.24 0 0.2" rpy="0 0 0" />
+        <origin xyz="0.22 0 0.2" rpy="0 0 0" />
     </joint>
     <!-- <xacro:rove_ros2_control/> -->

Commit message: Update rove.urdf.xacro

File: src/rove_description/urdf/rove.urdf.xacro (robot description, xacro)
@@ -20,5 +20,5 @@
             <origin xyz="0 0 0" rpy="0 0 0"/>
             <geometry>
-                <mesh filename="https://raw.githubusercontent.com/clubcapra/rove/main/src/rove_description/meshes/base.stl"/>
+                <mesh filename="file://$(find rove_description)/meshes/base.stl"/>
             </geometry>
             <material name="frame_color"/>

Commit message: Done merging live and main

File: src/rove_description/urdf/rove.urdf.xacro (robot description, xacro)
@@ -2,11 +2,11 @@
 <robot name="rove" xmlns:xacro="http://www.ros.org/wiki/xacro">
     <material name="rubber_color">
-        <color rgba="0.1 0.1 0.1 1.0"/>
+        <color rgba="0.1 0.1 0.1 1.0" />
     </material>
     <material name="frame_color">
-        <color rgba="0.5 0.5 0.5 1.0"/>
+        <color rgba="0.5 0.5 0.5 1.0" />
     </material>
     <material name="lidar_color">
-        <color rgba="1 0 0 1.0"/>
+        <color rgba="1 0 0 1.0" />
     </material>
     <xacro:include filename="$(find rove_description)/urdf/gazebo.urdf.xacro" />
@@ -18,38 +18,36 @@
     <link name="base_link">
         <visual>
-            <origin xyz="0 0 0" rpy="0 0 0"/>
+            <origin xyz="0 0 0" rpy="0 0 0" />
             <geometry>
-                <mesh filename="file://$(find rove_description)/meshes/base.stl"/>
+                <mesh filename="file://$(find rove_description)/meshes/base.stl" />
             </geometry>
-            <material name="frame_color"/>
+            <material name="frame_color" />
         </visual>
         <visual>
-            <origin xyz="0 0 0" rpy="0 0 0"/>
+            <origin xyz="0 0 0" rpy="0 0 0" />
             <geometry>
-                <mesh filename="file://$(find rove_description)/meshes/base.stl"/>
+                <mesh filename="file://$(find rove_description)/meshes/base.stl" />
             </geometry>
-            <material name="frame_color"/>
+            <material name="frame_color" />
         </visual>
         <collision>
-            <origin xyz="0 0 0" rpy="0 0 0"/>
+            <origin xyz="0 0 0" rpy="0 0 0" />
             <geometry>
-                <mesh filename="file://$(find rove_description)/meshes/base.stl"/>
+                <mesh filename="file://$(find rove_description)/meshes/base.stl" />
             </geometry>
         </collision>
         <inertial>
-            <origin xyz="0 0 0.5" rpy="0 0 0"/>
-            <mass value="80"/>
-            <inertia ixx="1"  ixy="0"  ixz="0" iyy="1" iyz="0" izz="1" />
+            <origin xyz="0 0 0.5" rpy="0 0 0" />
+            <mass value="80" />
+            <inertia ixx="1" ixy="0" ixz="0" iyy="1" iyz="0" izz="1" />
         </inertial>
     </link>
-    <!-- <xacro:rove_ros2_control/> -->
-     <!-- Put these at -1 to mock the motors if working without the motors -->
-    <!-- <xacro:odrive_control fl_id="21" rl_id="22" fr_id="23" rr_id="24"/> -->
-    <!-- TODO Fix rr Odrive, it keeps crashing the rest of the drives. IT has been disabled for now. -->
-    <xacro:odrive_control fl_id="21" rl_id="22" fr_id="23" rr_id="24"/>
+    <!-- Put these at -1 to mock the motors if working without the motors -->
+    <xacro:odrive_control fl_id="21" rl_id="22" fr_id="23" rr_id="24" />
     <!-- Insert ovis on top of rove -->
     <!-- <xacro:property name="robot_root" value="base_link" />
     <xacro:property name="ovis_robot_namespace" value="rove" />
     <xacro:property name="ovis_base_origin" value="-0.2 0 0.2" />
-    <xacro:ovis base_parent="${robot_root}" prefix="${ovis_robot_namespace}" joint_base_origin_xyz="${ovis_base_origin}" /> -->
+    <xacro:ovis base_parent="${robot_root}" prefix="${ovis_robot_namespace}"
+    joint_base_origin_xyz="${ovis_base_origin}" /> -->
 </robot>

File: src/rove_description/urdf/sensor.urdf.xacro (robot description, xacro)
@@ -6,15 +6,15 @@
         <parent link="base_link" />
         <child link="sensor_link" />
-        <origin xyz="-0.1 0 0.4" rpy="0 0 0" />
+        <origin xyz="-0.3 0 0.4" rpy="0 0 0" />
     </joint>
     <joint name="zed_camera_joint" type="fixed">
         <parent link="sensor_link" />
         <child link="zed_camera_link" />
-        <origin xyz="-0.1 0 0" rpy="0 0 0" />
+        <origin xyz="0.1 0 0" rpy="0 0 0" />
     </joint>
     <joint name="camera_joint" type="fixed">
         <parent link="sensor_link" />
         <child link="camera_link" />
-        <origin xyz="-0.1 0 0" rpy="${-pi/2} 0 ${-pi/2}" />
+        <origin xyz="0.1 0 0" rpy="-1.57 0 -1.57" />
     </joint>
     <link name="camera_link">
@@ -25,5 +25,5 @@
         <visual>
             <geometry>
-                <cylinder length="0.1" radius="0.1" />
+                <cylinder length="0.05" radius="0.05" />
             </geometry>
         </visual>
@@ -31,5 +31,5 @@
             <origin xyz="0 0 0" rpy="0 0 0" />
             <geometry>
-                <cylinder length="0.1" radius="0.1" />
+                <cylinder length="0.05" radius="0.05" />
             </geometry>
         </collision>
@@ -42,5 +42,5 @@
         <visual>
             <geometry>
-                <cylinder length="0.1" radius="0.1" />
+                <cylinder length="0.05" radius="0.05" />
             </geometry>
         </visual>
@@ -48,5 +48,5 @@
             <origin xyz="0 0 0" rpy="0 0 0" />
             <geometry>
-                <cylinder length="0.1" radius="0.1" />
+                <cylinder length="0.05" radius="0.05" />
             </geometry>
         </collision>
@@ -61,5 +61,5 @@
             <origin xyz="0 0 0" rpy="0 0 0" />
             <geometry>
-                <cylinder length="0.1" radius="0.1" />
+                <cylinder length="0.05" radius="0.05" />
             </geometry>
         </visual>
@@ -67,10 +67,10 @@
             <origin xyz="0 0 0" rpy="0 0 0" />
             <geometry>
-                <cylinder length="0.1" radius="0.1" />
+                <cylinder length="0.05" radius="0.05" />
             </geometry>
         </collision>
     </link>
     <xacro:velodyne_lidar name="velodyne" parent_link="base_link">
-        <origin xyz="0.0 0.0 0.4" rpy="0 0 ${-pi/2}" />
+        <origin xyz="-0.2 0.0 0.5" rpy="0 0 ${-pi/2}" />
     </xacro:velodyne_lidar>
     <gazebo reference="sensor_link">

Commit message: rove urdf duplicate hull fix

File: src/rove_description/urdf/rove.urdf.xacro (robot description, xacro)
@@ -17,11 +17,4 @@
     <!-- <xacro:include filename="$(find ovis_description)/urdf/ovis.urdf.xacro" /> -->
     <link name="base_link">
-        <visual>
-            <origin xyz="0 0 0" rpy="0 0 0" />
-            <geometry>
-                <mesh filename="file://$(find rove_description)/meshes/base.stl" />
-            </geometry>
-            <material name="frame_color" />
-        </visual>
         <visual>
             <origin xyz="0 0 0" rpy="0 0 0" />
